File: Hardware/L-Band Bridge/L-Band Bridge.kicad_sch (KiCad schematic)
At the start: 64 parts, among them J1 SMA, J2 SMA, J3 SMA, J4 SMA, J5 Conn_02x08_Odd_Even, J6 SMA, J7 Conn_01x02_Socket, U1 ADL5906, U2 MAPS-010163-TR0500, U3 HMC472ALP4E, U4 GALI-52, U5 ADL5906, U6 GALI-52, U7 ADE-17H+, U8 DBTC-17-5LX+, U9 DBTC-17-5LX+

Commit message: Working on BOM
Parts:
- removed R13, R7: 8.25, Resistor_SMD:R_1206_3216Metric, symbol Device:R_Small_US
- R8: value 143 -> 150; footprint Resistor_SMD:R_2010_5025Metric -> Resistor_SMD:R_2512_6332Metric; Digikey (none) -> A116012TR-ND
- R9: value 143 -> 150; footprint Resistor_SMD:R_2010_5025Metric -> Resistor_SMD:R_2512_6332Metric
Connections:
- net +12V: now also R8.2, R9.1
Other:
- note added: "A116012TR-ND"
- moved on the sheet: C18
Changed lines of the file:
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@@
   (junction (at 67.31 175.26) (diameter 0) (color 0 0 0 0)
   )
-  (junction (at 113.03 101.6) (diameter 0) (color 0 0 0 0)
+  (junction (at 125.095 100.965) (diameter 0) (color 0 0 0 0)
   )
   (junction (at 82.55 69.85) (diameter 0) (color 0 0 0 0)
@@
     (stroke (width 0) (type default))
   )
-  (wire (pts (xy 130.81 101.6) (xy 129.54 101.6))
+  (wire (pts (xy 125.095 100.965) (xy 130.81 100.965))
     (stroke (width 0) (type default))
   )
@@
     (stroke (width 0) (type default))
   )
-  (wire (pts (xy 113.03 101.6) (xy 124.46 101.6))
-    (stroke (width 0) (type default))
-  )
   (wire (pts (xy 240.03 22.86) (xy 242.57 22.86))
     (stroke (width 0) (type default))
@@
     (stroke (width 0) (type default))
   )
-  (wire (pts (xy 113.03 107.95) (xy 113.03 109.22))
+  (wire (pts (xy 125.095 107.315) (xy 125.095 108.585))
     (stroke (width 0) (type default))
   )
@@
     (stroke (width 0) (type default))
   )
-  (wire (pts (xy 149.86 22.86) (xy 153.67 22.86))
-    (stroke (width 0) (type default))
-  )
   (wire (pts (xy 88.9 97.79) (xy 88.9 99.06))
     (stroke (width 0) (type default))
@@
     (stroke (width 0) (type default))
   )
-  (wire (pts (xy 113.03 100.33) (xy 113.03 101.6))
+  (wire (pts (xy 125.095 99.695) (xy 125.095 100.965))
     (stroke (width 0) (type default))
   )
@@
     (stroke (width 0) (type default))
   )
-  (wire (pts (xy 130.81 96.52) (xy 130.81 101.6))
+  (wire (pts (xy 130.81 96.52) (xy 130.81 100.965))
     (stroke (width 0) (type default))
   )
@@
     (stroke (width 0) (type default))
   )
-  (wire (pts (xy 113.03 101.6) (xy 113.03 102.87))
+  (wire (pts (xy 125.095 100.965) (xy 125.095 102.235))
     (stroke (width 0) (type default))
   )
@@
     (stroke (width 0) (type default))
   )
-  (wire (pts (xy 143.51 22.86) (xy 144.78 22.86))
+  (wire (pts (xy 143.51 22.86) (xy 153.67 22.86))
     (stroke (width 0) (type default))
   )
@@
     (effects (font (size 1.27 1.27)) (justify left bottom))
   )
+  (text "A116012TR-ND" (at 131.445 98.425 0)
+    (effects (font (size 1.27 1.27)) (justify left bottom))
+  )
   (text "DC-DC Converter 12V to +5V and -5V\nRP-1205D\nOR\nPDQE10-Q24-D5-D"
     (at 25.4 115.57 0)
@@
     )
   )
-  (symbol (lib_id "Device:R_Small_US") (at 147.32 22.86 90) (unit 1)
-    (in_bom yes) (on_board yes) (dnp no) (fields_autoplaced)
-    (property "Reference" "R13" (at 147.32 17.78 90)
-      (effects (font (size 1.27 1.27)))
-    )
-    (property "Value" "8.25" (at 147.32 20.32 90)
-      (effects (font (size 1.27 1.27)))
-    )
-    (property "Footprint" "Resistor_SMD:R_1206_3216Metric" (at 147.32 22.86 0)
-      (effects (font (size 1.27 1.27)) hide)
-    )
-    (property "Datasheet" "~" (at 147.32 22.86 0)
-      (effects (font (size 1.27 1.27)) hide)
-    )
-    (pin "1")
-    (pin "2")
-    (instances
-      (project "L-Band Bridge"
-        (path "/ba7ea571-4dee-4705-9fa7-fb1d096b178c"
-          (reference "R13") (unit 1)
-        )
-      )
-    )
-  )
-  (symbol (lib_id "Device:C_Small") (at 113.03 105.41 180) (unit 1)
+  (symbol (lib_id "Device:C_Small") (at 125.095 104.775 180) (unit 1)
     (in_bom yes) (on_board yes) (dnp no)
-    (property "Reference" "C18" (at 116.84 105.41 0)
+    (property "Reference" "C18" (at 128.905 104.775 0)
       (effects (font (size 1.27 1.27)))
     )
-    (property "Value" "100nF" (at 117.475 103.505 0)
+    (property "Value" "100nF" (at 129.54 102.87 0)
       (effects (font (size 1.27 1.27)))
     )
-    (property "Footprint" "Capacitor_SMD:C_0402_1005Metric" (at 113.03 105.41 0)
+    (property "Footprint" "Capacitor_SMD:C_0402_1005Metric" (at 125.095 104.775 0)
       (effects (font (size 1.27 1.27)) hide)
     )
-    (property "Datasheet" "~" (at 113.03 105.41 0)
+    (property "Datasheet" "~" (at 125.095 104.775 0)
       (effects (font (size 1.27 1.27)) hide)
     )
@@
     )
   )
-  (symbol (lib_id "power:+12V") (at 113.03 100.33 0) (unit 1)
+  (symbol (lib_id "power:+12V") (at 125.095 99.695 0) (unit 1)
     (in_bom yes) (on_board yes) (dnp no) (fields_autoplaced)
-    (property "Reference" "#PWR026" (at 113.03 104.14 0)
+    (property "Reference" "#PWR026" (at 125.095 103.505 0)
       (effects (font (size 1.27 1.27)) hide)
     )
-    (property "Value" "+12V" (at 113.03 96.52 0)
+    (property "Value" "+12V" (at 125.095 95.885 0)
       (effects (font (size 1.27 1.27)))
     )
-    (property "Footprint" "" (at 113.03 100.33 0)
+    (property "Footprint" "" (at 125.095 99.695 0)
       (effects (font (size 1.27 1.27)) hide)
     )
-    (property "Datasheet" "" (at 113.03 100.33 0)
+    (property "Datasheet" "" (at 125.095 99.695 0)
       (effects (font (size 1.27 1.27)) hide)
     )
@@
     )
   )
-  (symbol (lib_id "power:GND") (at 113.03 109.22 0) (unit 1)
+  (symbol (lib_id "power:GND") (at 125.095 108.585 0) (unit 1)
     (in_bom yes) (on_board yes) (dnp no)
-    (property "Reference" "#PWR027" (at 113.03 115.57 0)
+    (property "Reference" "#PWR027" (at 125.095 114.935 0)
       (effects (font (size 1.27 1.27)) hide)
     )
-    (property "Value" "GND" (at 113.03 113.03 0)
+    (property "Value" "GND" (at 125.095 112.395 0)
       (effects (font (size 1.27 1.27)))
     )
-    (property "Footprint" "" (at 113.03 109.22 0)
+    (property "Footprint" "" (at 125.095 108.585 0)
       (effects (font (size 1.27 1.27)) hide)
     )
-    (property "Datasheet" "" (at 113.03 109.22 0)
+    (property "Datasheet" "" (at 125.095 108.585 0)
       (effects (font (size 1.27 1.27)) hide)
     )
@@
     )
   )
-  (symbol (lib_id "Device:R_Small_US") (at 127 101.6 90) (unit 1)
-    (in_bom yes) (on_board yes) (dnp no)
-    (property "Reference" "R7" (at 127 97.79 90)
-      (effects (font (size 1.27 1.27)))
-    )
-    (property "Value" "8.25" (at 127 99.695 90)
-      (effects (font (size 1.27 1.27)))
-    )
-    (property "Footprint" "Resistor_SMD:R_1206_3216Metric" (at 127 101.6 0)
-      (effects (font (size 1.27 1.27)) hide)
-    )
-    (property "Datasheet" "~" (at 127 101.6 0)
-      (effects (font (size 1.27 1.27)) hide)
-    )
-    (pin "1")
-    (pin "2")
-    (instances
-      (project "L-Band Bridge"
-        (path "/ba7ea571-4dee-4705-9fa7-fb1d096b178c"
-          (reference "R7") (unit 1)
-        )
-      )
-    )
-  )
   (symbol (lib_id "power:GND") (at 177.8 91.44 0) (unit 1)
     (in_bom yes) (on_board yes) (dnp no)
@@
       (effects (font (size 1.27 1.27)) (justify left))
     )
-    (property "Value" "143" (at 132.08 95.25 0)
+    (property "Value" "150" (at 132.08 95.25 0)
       (effects (font (size 1.27 1.27)) (justify left))
     )
-    (property "Footprint" "Resistor_SMD:R_2010_5025Metric" (at 130.81 93.98 0)
+    (property "Footprint" "Resistor_SMD:R_2512_6332Metric" (at 130.81 93.98 0)
+      (effects (font (size 1.27 1.27)) hide)
+    )
+    (property "Datasheet" "https://www.digikey.com/en/products/detail/te-connectivity-passive-product/3521150RFT/4279879" (at 130.81 93.98 0)
       (effects (font (size 1.27 1.27)) hide)
     )
-    (property "Datasheet" "~" (at 130.81 93.98 0)
+    (property "Digikey" "A116012TR-ND" (at 130.81 93.98 0)
       (effects (font (size 1.27 1.27)) hide)
     )
@@
       (effects (font (size 1.27 1.27)) (justify left))
     )
-    (property "Value" "143" (at 146.05 31.115 0)
+    (property "Value" "150" (at 146.05 31.115 0)
       (effects (font (size 1.27 1.27)) (justify left))
     )
-    (property "Footprint" "Resistor_SMD:R_2010_5025Metric" (at 143.51 29.21 0)
+    (property "Footprint" "Resistor_SMD:R_2512_6332Metric" (at 143.51 29.21 0)
       (effects (font (size 1.27 1.27)) hide)
     )
