File: Hardware/S-Band Transceiver/S-Band Transceiver.kicad_sch (KiCad schematic)
At the start: 26 parts, among them J1 SMA, U1 HMC8193, U2 HMC8193, U3 ADG901BCPZ, U4 GALI-39, U5 GALI-39, U6 GP2Y1+, U7 GALI-39, U8 YAT-10A+, U9 GALI-39

Commit message: Added receiver bypass switch comment
Parts:
- added C9: 100pF, symbol Device:C_Small
Other:
- note added: "ADRF5019BCPZN-R7 SPDT Switch for RX Bypass LNA"
Changed lines of the file:
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@@
 (kicad_sch (version 20230121) (generator eeschema)
   (paper "A4")
+  (text "ADRF5019BCPZN-R7\nSPDT Switch for RX Bypass LNA" (at 174.625 69.85 0)
+    (effects (font (size 1.27 1.27)) (justify left bottom))
+  )
   (symbol (lib_id "Device:R_Small_US") (at 239.395 25.4 0) (unit 1)
     (in_bom yes) (on_board yes) (dnp no) (fields_autoplaced)
@@
         )
       )
+    )
+  )
+  (symbol (lib_id "Device:C_Small") (at 284.48 36.83 90) (unit 1)
+    (in_bom yes) (on_board yes) (dnp no)
+    (property "Reference" "C9" (at 284.48 41.91 90)
+      (effects (font (size 1.27 1.27)))
+    )
+    (property "Value" "100pF" (at 284.48 40.005 90)
+      (effects (font (size 1.27 1.27)))
+    )
+    (property "Footprint" "" (at 284.48 36.83 0)
+      (effects (font (size 1.27 1.27)) hide)
+    )
+    (property "Datasheet" "~" (at 284.48 36.83 0)
+      (effects (font (size 1.27 1.27)) hide)
+    )
+    (pin "1")
+    (pin "2")
+    (instances
+      (project "S-Band Transceiver"
+        (path "/811f57cf-e3df-4fba-aff9-353adc85299e"
+          (reference "C9") (unit 1)
+        )
+      )
