File: Hardware/S-Band Transceiver/S-Band Transceiver.kicad_sch (KiCad schematic)
At the start: 27 parts, among them J1 SMA, U1 HMC8193, U2 HMC8193, U3 ADG901BCPZ, U4 GALI-39, U5 GALI-39, U6 GP2Y1+, U7 GALI-39, U8 YAT-10A+, U9 GALI-39

Commit message: Updates to Schematic
Parts:
- removed U8: YAT-10A+, symbol _tim-RF:YAT-10A+
Other:
- added sheet Microcontroller (micro.kicad_sch)
- added sheet Power Supply (power_supply.kicad_sch)
- added sheet Receiver (receiver.kicad_sch)
- added sheet Synthesizer (synthesizer.kicad_sch)
- added sheet Transmitter (transmitter.kicad_sch)
- moved on the sheet: C1, C2, C3, C4, C5, C6, C7, C8, C9, J1, L1, L2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

Commit message: Updating schematic
Other:
- note added: "DIRECTIONAL COUPLER DCW-22-332+"
Changed lines of the file:
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@@
+		)
+	)
+	(text "DIRECTIONAL COUPLER\nDCW-22-332+\n"
+		(exclude_from_sim no)
+		(at 191.77 110.49 0)
+		(effects
+			(font
+				(size 1.27 1.27)
+			)
 		)
 	)

Commit message: Updates to schematic
Changed lines of the file:
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@@
 	(generator_version "8.0")
 	(paper "A4")
-	(text_box "Low Cost Solution:\nDesign must cost < $200\nNo IQ Mixer, phase shifter PE44820\nDirectional coupler: D17W+\nLog Det: ADL5906\nSplitter: GP2Y1+\nAtten: DAT-31A+\nIQ Mixer: ADL5380\nAMP: SKY65017-70LF\nSynth: ADF4351\n\n\n\n\n\n"
+	(text_box "Low Cost Solution:\nDesign must cost < $200\nNo IQ Mixer, phase shifter PE44820\nDirectional coupler: D17W+ or DCW-22-332+\nLog Det: ADL5906\nSplitter: GP2Y1+\nAtten: DAT-31A+\nIQ Mixer: ADL5380\nAMP: SKY65017-70LF\nSynth: ADF4351\n\n\n\n\n\n"
 		(exclude_from_sim no)
 		(at 217.17 135.89 0)

Commit message: Updating schematic
Parts:
- removed C1, C2, C3, C4, C5, C6, C7, C8, C9: 100pF, symbol Device:C_Small
- removed J1: SMA, symbol Connector:Conn_Coaxial
- removed L1, L2, L3, L4: 120nH, symbol Device:L_Small
- removed R1, R2, R3, R4: 100*, symbol Device:R_Small_US
- removed U1, U2: HMC8193, symbol _tim-RF:HMC8193
- removed U3: ADG901BCPZ, Package_CSP:LFCSP-8-1EP_3x3mm_P0.5mm_EP1.45x1.74mm, symbol RF_Switch:ADG901BCPZ
- removed U4, U5, U7, U9: GALI-39, Package_TO_SOT_SMD:SOT-89-3, symbol RF_Amplifier:GALI-39
- removed U6: GP2Y1+, symbol _tim-RF:GP2Y1+
Other:
- note removed: "ADRF5019BCPZN-R7 SPDT Switch for RX Bypass LNA"
