File: Hardware/S-Band Transceiver/S-Band Transceiver.kicad_sch (KiCad schematic)
At the start: 0 parts

Commit message: Updating board layout and routing
Parts:
- added H1, H2, H3, H4: 4-40, B12T_MountingHole:4-40_Hole_Pad, symbol Mechanical:MountingHole_Pad
Connections:
- new net GND: H1.1, H2.1, H3.1, H4.1

Commit message: Minor Changes
Other:
- note added: "Updates: Add 2nd synthesizer Remove Digital phase shifter"
Changed lines of the file:
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@@
+		)
+	)
+	(text "Updates:\nAdd 2nd synthesizer\nRemove Digital phase shifter\n"
+		(exclude_from_sim no)
+		(at 151.892 20.828 0)
+		(effects
+			(font
+				(size 1.27 1.27)
+			)
+			(justify left)
 		)
 	)
