File: Hardware/S-Band Transceiver/_autosave-S-Band Transceiver.kicad_pcb (KiCad board)
At the start: 4 copper layers, 171.4 x 101.6 mm, 216 parts, among them J1 SMA, J2 SMA, J3 AVR-UPDI-6, J4 USB_C_Receptacle_USB2.0_16P, J5 SMA, J6 SMA, J7 SMA, J8 SMA, SW1 SW_Push, U1 ADF4351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

Commit message: Routing board
Routing:
- net Net-(U7-RFOUT): track 0.00 -> 3.52 mm
- net Net-(U8-RF1): track 0.00 -> 3.17 mm
Changed lines of the file:
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@@
 		(start 130.054999 62.1538)
 		(end 126.3492 62.1538)
-		(width 0.25)
+		(width 0.394208)
 		(layer "F.Cu")
 		(net 16)
@@
 		(start 130.5986 61.2902)
 		(end 130.5986 61.610199)
-		(width 0.25)
+		(width 0.394208)
 		(layer "F.Cu")
 		(net 16)
@@
 		(start 130.5986 61.610199)
 		(end 130.054999 62.1538)
-		(width 0.25)
+		(width 0.394208)
 		(layer "F.Cu")
 		(net 16)
@@
 		(start 125.3892 62.1538)
 		(end 124.2206 62.1538)
-		(width 0.25)
+		(width 0.394208)
 		(layer "F.Cu")
 		(net 17)
@@
 		(start 124.2206 62.1538)
 		(end 124.1698 62.2046)
-		(width 0.25)
+		(width 0.394208)
 		(layer "F.Cu")
 		(net 17)
@@
 		(start 130.5428 62.8372)
 		(end 130.388 62.992)
-		(width 0.25)
+		(width 0.394208)
 		(layer "F.Cu")
 		(net 18)
@@
 		(start 130.388 62.992)
 		(end 126.6286 62.992)
-		(width 0.25)
+		(width 0.394208)
 		(layer "F.Cu")
 		(net 18)
@@
 		(start 126.6286 62.992)
 		(end 126.3492 63.2714)
-		(width 0.25)
+		(width 0.394208)
 		(layer "F.Cu")
 		(net 18)
@@
 		(start 125.3892 63.2714)
 		(end 124.2206 63.2714)
-		(width 0.25)
+		(width 0.394208)
 		(layer "F.Cu")
 		(net 19)
@@
 		(start 124.2206 63.2714)
 		(end 124.1698 63.3222)
-		(width 0.25)
+		(width 0.394208)
 		(layer "F.Cu")
 		(net 19)
@@
 	)
 	(segment
+		(start 94.181 114.316)
+		(end 94.73271 114.316)
+		(width 0.254)
+		(layer "F.Cu")
+		(net 28)
+	)
+	(segment
+		(start 94.73271 114.316)
+		(end 94.75391 114.3372)
+		(width 0.254)
+		(layer "F.Cu")
+		(net 28)
+	)
+	(segment
+		(start 97.338 114.3372)
+		(end 94.75391 114.3372)
+		(width 0.394208)
+		(layer "F.Cu")
+		(net 28)
+	)
+	(segment
+		(start 98.298 114.3372)
+		(end 101.20409 114.3372)
+		(width 0.394208)
+		(layer "F.Cu")
+		(net 29)
+	)
+	(segment
+		(start 101.8055 114.3)
+		(end 101.24129 114.3)
+		(width 0.254)
+		(layer "F.Cu")
+		(net 29)
+	)
+	(segment
+		(start 101.24129 114.3)
+		(end 101.20409 114.3372)
+		(width 0.254)
+		(layer "F.Cu")
+		(net 29)
+	)
+	(segment
