File: Hardware/S-Band Transceiver/micro.kicad_sch (KiCad schematic)
At the start: 46 parts, among them J3 AVR-UPDI-6, J4 USB_C_Receptacle_USB2.0_16P, SW1 SW_Push, U2 AVR128DA48x-xPT, U3 ADS1118IDGS, U4 FT231XQ

Commit message: Updating BOM
Other:
- note added: "Should shield be grounded?"
Changed lines of the file:
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@@
+		)
+	)
+	(text "Should shield be grounded?"
+		(exclude_from_sim no)
+		(at 181.356 74.93 0)
+		(effects
+			(font
+				(size 1.27 1.27)
+			)
 		)
 	)
