File: Hardware/Bridge Controller/Bridge_Controller/DAQ.kicad_sch (KiCad schematic)
At the start: 64 parts, among them J10 SMA-J-P-H-ST-EM1, J5 SMA-J-P-H-ST-EM1, J6 SMA-J-P-H-ST-EM1, J7 SMA-J-P-H-ST-EM1, J8 SMA-J-P-H-ST-EM1, J9 SMA-J-P-H-ST-EM1, U10 LMV358, U11 LMV358, U12 MCP1501-25xCH, U6 ADS1118IDGS, U7 AD9833xRM, U8 LMV358, U9 DAC8532, X1 XO32

Commit message: Updates to DAQ board layout
Parts:
- added C31, C32, C33, C34: 100nF, Capacitor_SMD:C_0603_1608Metric, symbol Device:C_Small
- added R45: 27, Resistor_SMD:R_0603_1608Metric, symbol Device:R_Small_US
- C17: renamed from C31; footprint Capacitor_SMD:C_0402_1005Metric -> Capacitor_SMD:C_0603_1608Metric
- C18: renamed from C22; footprint (none) -> Capacitor_SMD:C_0603_1608Metric
- C19: renamed from C21; footprint (none) -> Capacitor_SMD:C_0603_1608Metric
- C20: renamed from C32; footprint Capacitor_SMD:C_0402_1005Metric -> Capacitor_SMD:C_0603_1608Metric
- C21: renamed from C28; footprint (none) -> Capacitor_SMD:C_0603_1608Metric
- C22: renamed from C26; footprint (none) -> Capacitor_SMD:C_0603_1608Metric
- C23: renamed from C30; footprint (none) -> Capacitor_SMD:C_0603_1608Metric
- C24: renamed from C27; footprint (none) -> Capacitor_SMD:C_0603_1608Metric
- C25: renamed from C29; footprint (none) -> Capacitor_SMD:C_0603_1608Metric
- C26: renamed from C19; footprint (none) -> Capacitor_SMD:C_0603_1608Metric
- C27: renamed from C20; footprint (none) -> Capacitor_SMD:C_0603_1608Metric
- C28: renamed from C23; footprint (none) -> Capacitor_SMD:C_0603_1608Metric
- C29: renamed from C24; footprint (none) -> Capacitor_SMD:C_0603_1608Metric
- C30: renamed from C25; footprint (none) -> Capacitor_SMD:C_0603_1608Metric
- J5: renamed from J10; footprint Connector_Coaxial:SMA_Samtec_SMA-J-P-X-ST-EM1_EdgeMount -> Connector_Coaxial:SMA_Amphenol_132291_Vertical
- R16: renamed from R57; footprint (none) -> Resistor_SMD:R_0603_1608Metric
- R19: renamed from R48; footprint (none) -> Resistor_SMD:R_0603_1608Metric
- R20: renamed from R49; footprint (none) -> Resistor_SMD:R_0603_1608Metric
- R21: renamed from R58; footprint (none) -> Resistor_SMD:R_0603_1608Metric
- R22: renamed from R59; footprint (none) -> Resistor_SMD:R_0603_1608Metric
- R23: renamed from R60; footprint (none) -> Resistor_SMD:R_0603_1608Metric
- R24: renamed from R51; footprint (none) -> Resistor_SMD:R_0603_1608Metric
- R25: renamed from R50; footprint (none) -> Resistor_SMD:R_0603_1608Metric
- R26: renamed from R55; footprint (none) -> Resistor_SMD:R_0603_1608Metric
- R27: renamed from R32; footprint (none) -> Resistor_SMD:R_0603_1608Metric
- R28: renamed from R52; footprint (none) -> Resistor_SMD:R_0603_1608Metric
- R29: renamed from R33; footprint (none) -> Resistor_SMD:R_0603_1608Metric
- R30: renamed from R34; footprint (none) -> Resistor_SMD:R_0603_1608Metric
- R31: renamed from R35; footprint (none) -> Resistor_SMD:R_0603_1608Metric
- R32: renamed from R37; footprint (none) -> Resistor_SMD:R_0603_1608Metric
- R33: renamed from R36; footprint (none) -> Resistor_SMD:R_0603_1608Metric
- R34: renamed from R38; footprint (none) -> Resistor_SMD:R_0603_1608Metric
- R35: renamed from R56; footprint (none) -> Resistor_SMD:R_0603_1608Metric
- R36: renamed from R39; footprint (none) -> Resistor_SMD:R_0603_1608Metric
- R38: renamed from R40; footprint (none) -> Resistor_SMD:R_0603_1608Metric
- R39: renamed from R41; footprint (none) -> Resistor_SMD:R_0603_1608Metric
- R40: renamed from R44; footprint (none) -> Resistor_SMD:R_0603_1608Metric
- R41: renamed from R43; footprint (none) -> Resistor_SMD:R_0603_1608Metric
- R42: renamed from R54; footprint (none) -> Resistor_SMD:R_0603_1608Metric
- R43: renamed from R46; footprint (none) -> Resistor_SMD:R_0603_1608Metric
- R44: renamed from R47; footprint (none) -> Resistor_SMD:R_0603_1608Metric
- TP1: renamed from TP6; footprint (none) -> TestPoint:TestPoint_Pad_D1.0mm
- TP2: renamed from TP5; footprint (none) -> TestPoint:TestPoint_Pad_D1.0mm
- TP3: renamed from TP4; footprint (none) -> TestPoint:TestPoint_Pad_D1.0mm
- TP4: renamed from TP7; footprint (none) -> TestPoint:TestPoint_Pad_D1.0mm
- TP5: renamed from TP1; footprint (none) -> TestPoint:TestPoint_Pad_D1.0mm
- TP6: renamed from TP3; footprint (none) -> TestPoint:TestPoint_Pad_D1.0mm
- TP7: renamed from TP2; footprint (none) -> TestPoint:TestPoint_Pad_D1.0mm
- U5: renamed from U10; footprint (none) -> Package_SO:VSSOP-8_3.0x3.0mm_P0.65mm
- U6: renamed from U11; footprint (none) -> Package_SO:VSSOP-8_3.0x3.0mm_P0.65mm
- U8: footprint (none) -> Package_SO:VSSOP-8_3.0x3.0mm_P0.65mm
- U9: renamed from U6; footprint (none) -> Package_SO:VSSOP-10_3x3mm_P0.5mm
- X1: value XO32 -> XO53; footprint Oscillator:Oscillator_SMD_EuroQuartz_XO32-4Pin_3.2x2.5mm -> Oscillator:Oscillator_SMD_EuroQuartz_XO53-4Pin_5.0x3.2mm; Digikey (none) -> XC1902CT-ND
- renumbered J6 to J10, J9 to J6, J8 to J7, J7 to J8, J5 to J9, R42 to R17, R45 to R18, R53 to R37, U9 to U3, U7 to U4, U12 to U7
Connections:
- net +5V: now also C31.2, C32.1
- net GND: now also C31.1, C32.2, C33.1, C34.2
- net at U6.1, U6.2 (-): now also R45.2; no longer C21.1
- net at U4.1 (COMP): now also C34.1
- net at U4.3 (CAP/2.5V): now also C33.2
- new net: C21.1, R45.1
Other:
- company: (none) -> openEPR
- title: (none) -> openEPR DAQ
- moved on the sheet: C21, J6, TP4

Commit message: Routing Board
Parts:
- added C35: 100nF, Capacitor_SMD:C_0603_1608Metric, symbol Device:C_Small
Connections:
- net +5V: now also C35.2
- net GND: now also U9.3 (GND), C35.1
- net at C20.1, R21.2, U6.3 (+): now also TP4.1
- net at C21.2, J6.1 (In): no longer TP4.1
Other:
- moved on the sheet: TP4

Commit message: Finalizing Board Routing
Parts:
- renumbered C31 to C18, C33 to C19, C32 to C20, C34 to C21, C18 to C22, C19 to C23, C20 to C24, C21 to C25, C22 to C26, C23 to C27, C24 to C28, C25 to C29, C26 to C30, C27 to C31, C28 to C32, C35 to C33, C29 to C34, C30 to C35, J9 to J10, J10 to J11, J5 to J6, J6 to J7, J7 to J8, J8 to J9, R16 to R19, R17 to R20, R18 to R21, R19 to R22, R20 to R23, R21 to R24, R22 to R25, R23 to R26, R24 to R27, R25 to R28, R45 to R29, R26 to R30, R27 to R31, R28 to R32, R29 to R33, R30 to R34, R31 to R35, R32 to R36, R33 to R37, R34 to R38, R35 to R39, R36 to R40, R37 to R41, R38 to R42, R39 to R43, R40 to R44, R41 to R45, R42 to R46, R43 to R47, R44 to R48, TP4 to TP2, TP2 to TP3, TP3 to TP4

Commit message: Updating BOM
Parts:
- C17, C18, C19, C20, C21, C22, C23, C25, C26, C27, C28, C29, C30, C31, C32, C33, C34, C35: Digikey (none) -> 490-4779-1-ND
- C24: Digikey (none) -> 490-4944-1-ND
- J6: value SMA-J-P-H-ST-EM1 -> 132291
- R19, R22, R23, R24, R25, R26, R30, R31, R32, R33, R36, R37, R38, R40, R42, R43, R44, R45, R46, R47, R48: Digikey (none) -> 311-10.0KHRCT-ND
- R20, R21: value 0 -> 27; Digikey (none) -> 311-27GRCT-ND
- R27, R28: value 1k -> 27; Digikey (none) -> 311-27GRCT-ND
- R29: Digikey (none) -> 311-27GRCT-ND
- R34, R35, R39, R41: Digikey (none) -> 311-1.00KHRCT-ND
- U4: Digikey (none) -> 505-AD9833BRMZ-ND
- U5, U6, U8: Digikey (none) -> 296-18457-1-ND
- U9: Digikey (none) -> 296-38850-1-ND

Commit message: Minor Updates to Board
Connections:
- net at C22.1, R22.2, U5.3 (+): now also TP3.1
- net at J8.1 (In), R27.2: no longer TP3.1
- net at J9.1 (In), R28.2: no longer TP4.1
- net at C23.1, R23.2, U5.5 (+): now also TP4.1
Other:
- moved on the sheet: TP3, TP4
Changed lines of the file:
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@@
 	)
 	(junction
+		(at 76.2 154.94)
+		(diameter 0)
+		(color 0 0 0 0)
+	)
+	(junction
 		(at 186.69 38.1)
 		(diameter 0)
@@
 	)
 	(junction
+		(at 76.2 139.7)
+		(diameter 0)
+		(color 0 0 0 0)
+	)
+	(junction
 		(at 186.69 78.74)
 		(diameter 0)
@@
 	)
 	(junction
-		(at 107.95 142.24)
-		(diameter 0)
-		(color 0 0 0 0)
-	)
-	(junction
 		(at 44.45 137.16)
 		(diameter 0)
@@
 	)
 	(junction
-		(at 107.95 157.48)
-		(diameter 0)
-		(color 0 0 0 0)
-	)
-	(junction
 		(at 236.22 40.64)
 		(diameter 0)
@@
 	(wire
 		(pts
-			(xy 107.95 157.48) (xy 118.11 157.48)
-		)
-		(stroke
-			(width 0)
-			(type default)
-		)
-	)
-	(wire
-		(pts
 			(xy 186.69 38.1) (xy 186.69 39.37)
 		)
@@
 	(wire
 		(pts
+			(xy 76.2 139.7) (xy 80.01 139.7)
+		)
+		(stroke
+			(width 0)
+			(type default)
+		)
+	)
+	(wire
+		(pts
 			(xy 205.74 139.7) (xy 205.74 140.97)
 		)
@@
 	(wire
 		(pts
+			(xy 76.2 154.94) (xy 80.01 154.94)
+		)
+		(stroke
+			(width 0)
+			(type default)
+		)
+	)
+	(wire
+		(pts
 			(xy 274.32 132.08) (xy 274.32 133.35)
 		)
@@
 	(wire
 		(pts
-			(xy 107.95 140.97) (xy 107.95 142.24)
+			(xy 76.2 138.43) (xy 76.2 139.7)
 		)
 		(stroke
@@
 	(wire
 		(pts
-			(xy 107.95 156.21) (xy 107.95 157.48)
+			(xy 76.2 153.67) (xy 76.2 154.94)
 		)
 		(stroke
@@
 	(wire
 		(pts
-			(xy 107.95 142.24) (xy 118.11 142.24)
-		)
-		(stroke
-			(width 0)
-			(type default)
-		)
-	)
-	(wire
-		(pts
 			(xy 66.04 64.77) (xy 62.23 64.77)
 		)
@@
 	(wire
 		(pts
-			(xy 69.85 154.94) (xy 80.01 154.94)
+			(xy 69.85 154.94) (xy 76.2 154.94)
 		)
 		(stroke
@@
 	(wire
 		(pts
-			(xy 69.85 139.7) (xy 80.01 139.7)
+			(xy 69.85 139.7) (xy 76.2 139.7)
 		)
 		(stroke
@@
 	(wire
 		(pts
-			(xy 104.14 157.48) (xy 107.95 157.48)
+			(xy 104.14 157.48) (xy 118.11 157.48)
 		)
 		(stroke
@@
 	(wire
 		(pts
-			(xy 104.14 142.24) (xy 107.95 142.24)
+			(xy 104.14 142.24) (xy 118.11 142.24)
 		)
 		(stroke
@@
 	(symbol
 		(lib_id "Connector:TestPoint")
-		(at 107.95 140.97 0)
+		(at 76.2 138.43 0)
 		(unit 1)
 		(exclude_from_sim no)
@@
 		(dnp no)
 		(property "Reference" "TP3"
-			(at 106.68 137.668 0)
+			(at 74.93 135.128 0)
 			(effects
 				(font
@@
 		)
 		(property "Value" "TestPoint"
-			(at 114.3 135.128 0)
+			(at 82.55 132.588 0)
 			(effects
 				(font
@@
 		)
 		(property "Footprint" "TestPoint:TestPoint_Pad_D1.0mm"
-			(at 113.03 140.97 0)
+			(at 81.28 138.43 0)
 			(effects
 				(font
@@
 		)
 		(property "Datasheet" "~"
-			(at 113.03 140.97 0)
+			(at 81.28 138.43 0)
 			(effects
 				(font
@@
 		)
 		(property "Description" "test point"
-			(at 107.95 140.97 0)
+			(at 76.2 138.43 0)
 			(effects
 				(font
@@
 	(symbol
 		(lib_id "Connector:TestPoint")
-		(at 107.95 156.21 0)
+		(at 76.2 153.67 0)
 		(unit 1)
 		(exclude_from_sim no)
@@
 		(dnp no)
 		(property "Reference" "TP4"
-			(at 106.68 152.908 0)
+			(at 74.93 150.368 0)
 			(effects
 				(font
@@
 		)
 		(property "Value" "TestPoint"
-			(at 114.3 150.368 0)
+			(at 82.55 147.828 0)
 			(effects
 				(font
@@
 		)
 		(property "Footprint" "TestPoint:TestPoint_Pad_D1.0mm"
-			(at 113.03 156.21 0)
+			(at 81.28 153.67 0)
 			(effects
 				(font
@@
 		)
 		(property "Datasheet" "~"
-			(at 113.03 156.21 0)
+			(at 81.28 153.67 0)
 			(effects
 				(font
@@
 		)
 		(property "Description" "test point"
-			(at 107.95 156.21 0)
+			(at 76.2 153.67 0)
 			(effects
 				(font

Commit message: Adding gerbers
Parts:
- J6: value 132291 -> 2057-RF2-19A-T-00-50-G-ND; Digikey SAM8857-ND -> 2057-RF2-19A-T-00-50-G-ND
Changed lines of the file:
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@@
 			)
 		)
-		(property "Value" "132291"
+		(property "Value" "2057-RF2-19A-T-00-50-G-ND"
 			(at 78.74 99.3531 0)
 			(effects
@@
 			)
 		)
-		(property "Digikey" "SAM8857-ND"
+		(property "Digikey" "2057-RF2-19A-T-00-50-G-ND"
 			(at 76.2 97.79 0)
 			(effects

Commit message: Updating DAQ board schematic
Parts:
- added C36: 100nF, Capacitor_SMD:C_0603_1608Metric, symbol Device:C_Small
- added R49, R50, R51, R52: 10k, Resistor_SMD:R_0603_1608Metric, symbol Device:R_Small_US
Connections:
- net +2V5: now also C18.2, U3.2 (VREF)
- net +5V: now also C36.1; no longer C18.2, U3.2 (VREF)
- net GND: now also C36.2, R51.1, R52.1
- net at R27.1, U5.1: now also R50.2; no longer U5.2 (-)
- net at R28.1, U5.7: now also R49.2; no longer U5.6 (-)
- new net: R50.1, R51.2, U5.2 (-)
- new net: R49.1, R52.2, U5.6 (-)
Other:
- note added: "2725-B0509XT-2WR3-ND B0509XT-2WR3 DC DC CONVERTER 9V 2W Isolated Module DC DC Converter 1 Output 9V 222mA 4.5V - 5.5V Input"
- note added: "LDO Options: ADP7105 or ADP7102 or ADP7104"
- moved on the sheet: C22, C23, J8, J9, R22, R27, R28, TP3, TP4, U5A, U5B

Commit message: Updates to DAQ
Parts:
- C29, C30, C31: value 100nF -> 1uF
Changed lines of the file:
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@@
 			)
 		)
-		(property "Value" "100nF"
-			(at 209.296 146.812 0)
+		(property "Value" "1uF"
+			(at 210.312 145.034 0)
 			(effects
 				(font
@@
 			)
 		)
-		(property "Value" "100nF"
+		(property "Value" "1uF"
 			(at 229.87 45.7262 0)
 			(effects
@@
 			)
 		)
-		(property "Value" "100nF"
+		(property "Value" "1uF"
 			(at 229.87 86.3662 0)
 			(effects
