File: Hardware/Bridge Controller/Bridge_Controller/Bridge_Controller.kicad_pcb (KiCad board)
At the start: 2 copper layers, 58.4 x 99.1 mm, 119 parts, among them J1 AVR-UPDI-6, J10 SMA-J-P-H-ST-EM1, J2 Conn_02x08_standard_header_fo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, J3 Conn_02x08_standard_header_fo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, J4 USB_C_Receptacle_USB2.0_16P, J5 SMA-J-P-H-ST-EM1, J6 SMA-J-P-H-ST-EM1, J7 SMA-J-P-H-ST-EM1, J8 SMA-J-P-H-ST-EM1, J9 SMA-J-P-H-ST-EM1, SW1 SW_Push, U1 AVR128DA64x-xPT, U2 FT231XQ, U3 DAC8532, U4 AD9833xRM, U5 LMV358, U6 LMV358, U7 MCP1501-25xCH, U8 LMV358, U9 ADS1118IDGS, X1 XO53

Commit message: Routing Board
Parts:
- added C35: 100nF, Capacitor_SMD:C_0603_1608Metric, F.Cu at (64.1, 34.9)
- L1: value MH1608-601Y -> 10uH; footprint Inductor_SMD:L_0603_1608Metric -> Inductor_SMD:L_0805_2012Metric
- moved TP1 105.9 mm to (47.6, 91.4)
- moved R16 92.0 mm to (36.8, 97.8), turned to 180 degrees
- moved C17 90.7 mm to (38.7, 90.8), turned to 90 degrees
- moved R17 82.9 mm to (41.9, 91.4)
- moved R18 80.7 mm to (41.9, 89.5)
- moved TP7 24.4 mm to (50.8, 43.2)
- moved R23 19.0 mm to (38.1, 104.8)
- moved TP6 18.8 mm to (50.8, 33.7)
- moved TP4 18.3 mm to (34.3, 108.6)
- moved R42 16.9 mm to (64.1, 38.7)
- moved C25 16.5 mm to (64.1, 36.8)
- moved R22 14.6 mm to (38.1, 106.7)
- moved C18 11.6 mm to (29.2, 75.6), turned to 180 degrees
- moved R19 11.6 mm to (29.2, 73.7), turned to 0 degrees
- moved C1 10.8 mm to (40.6, 56.5)
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Connections:
- TP4 pad 1: Net-(J6-In) -> Net-(U6A-+)
- U9 pad 3: unconnected-(U9-GND-Pad3) -> GND
Routing:
- net SCLK: track 0.00 -> 78.5 mm, vias 0 -> 4
- net MOSI: track 0.00 -> 72.4 mm, vias 0 -> 4
- net AIN1: track 0.00 -> 66.8 mm, vias 0 -> 1
- net AIN0: track 0.00 -> 62.6 mm, vias 0 -> 1
- net ~{CS_ADC}: track 0.00 -> 62.4 mm, vias 0 -> 2
- net MISO: track 0.00 -> 61.8 mm, vias 0 -> 2
- net PG7: track 0.00 -> 59.3 mm, vias 0 -> 1
- net PG6: track 0.00 -> 57.5 mm, vias 0 -> 1
- net PG5: track 0.00 -> 54.7 mm, vias 0 -> 1
- net PG4: track 0.00 -> 51.5 mm, vias 0 -> 1
- net +5V: track 20.9 -> 69.6 mm, vias 0 -> 22
- net PG2: track 0.00 -> 47.3 mm, vias 0 -> 1
- net +2V5: track 0.00 -> 47.1 mm, vias 0 -> 2
- net PG3: track 0.00 -> 46.0 mm, vias 0 -> 1
- net PG0: track 0.00 -> 43.7 mm, vias 0 -> 1
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- added copper zone on In2.Cu, net +5V
- added copper zone on B.Cu, net GND
- added copper zone on F.Cu, net GND
- added copper zone on In1.Cu, net GND
Other:
- copper layers 2 -> 4
- board text added: "+2.5V"
- board text added: "ADC0"
- board text added: "ADC1"
- board text added: "DAC0"
- board text added: "DAC1"
- board text added: "DDS"
- board text added: "EXT CLK"
- board text added: "RESET"

Commit message: Fixed DRC errors on Board
Routing:
- net GND: track 30.9 -> 32.1 mm, vias 24 -> 41
- net ~{CS_DDS}: vias 1 -> 0
Changed lines of the file:
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@@
 	)
 	(segment
+		(start 55.372 84.53734)
+		(end 54.520678 85.388662)
+		(width 0.254)
+		(layer "F.Cu")
+		(net 1)
+	)
+	(segment
 		(start 65.003536 79.855551)
 		(end 64.227 80.632087)
@@
 	)
 	(via
+		(at 65.405 102.235)
+		(size 0.6)
+		(drill 0.3)
+		(layers "F.Cu" "B.Cu")
+		(free yes)
+		(net 1)
+	)
+	(via
+		(at 55.245 89.535)
+		(size 0.6)
+		(drill 0.3)
+		(layers "F.Cu" "B.Cu")
+		(free yes)
+		(net 1)
+	)
+	(via
 		(at 47.625 93.98)
 		(size 0.6)
@@
 	)
 	(via
+		(at 79.375 86.36)
+		(size 0.6)
+		(drill 0.3)
+		(layers "F.Cu" "B.Cu")
+		(free yes)
+		(net 1)
+	)
+	(via
+		(at 58.42 52.705)
+		(size 0.6)
+		(drill 0.3)
+		(layers "F.Cu" "B.Cu")
+		(free yes)
+		(net 1)
+	)
+	(via
 		(at 60.452 86.741)
 		(size 0.6)
@@
 	)
 	(via
+		(at 40.64 66.04)
+		(size 0.6)
+		(drill 0.3)
+		(layers "F.Cu" "B.Cu")
+		(free yes)
+		(net 1)
+	)
+	(via
 		(at 24.765 70.485)
 		(size 0.6)
@@
 	)
 	(via
+		(at 41.275 50.165)
+		(size 0.6)
+		(drill 0.3)
+		(layers "F.Cu" "B.Cu")
+		(free yes)
+		(net 1)
+	)
+	(via
 		(at 24.765 76.2)
 		(size 0.6)
@@
 	)
 	(via
+		(at 41.275 85.09)
+		(size 0.6)
+		(drill 0.3)
+		(layers "F.Cu" "B.Cu")
+		(free yes)
+		(net 1)
+	)
+	(via
 		(at 24.765 95.25)
 		(size 0.6)
@@
 	)
 	(via
+		(at 68.58 86.36)
+		(size 0.6)
+		(drill 0.3)
+		(layers "F.Cu" "B.Cu")
+		(free yes)
+		(net 1)
+	)
+	(via
 		(at 69.342 77.216)
 		(size 0.6)
@@
 	)
 	(via
+		(at 41.275 80.01)
+		(size 0.6)
+		(drill 0.3)
+		(layers "F.Cu" "B.Cu")
+		(free yes)
+		(net 1)
+	)
+	(via
 		(at 24.765 88.9)
 		(size 0.6)
@@
 	)
 	(via
+		(at 75.565 104.775)
+		(size 0.6)
+		(drill 0.3)
+		(layers "F.Cu" "B.Cu")
+		(free yes)
+		(net 1)
+	)
+	(via
+		(at 41.275 109.855)
+		(size 0.6)
+		(drill 0.3)
+		(layers "F.Cu" "B.Cu")
+		(free yes)
+		(net 1)
+	)
+	(via
 		(at 48.26 36.703)
 		(size 0.6)
@@
 	)
 	(via
+		(at 34.925 55.245)
+		(size 0.6)
+		(drill 0.3)
+		(layers "F.Cu" "B.Cu")
+		(free yes)
+		(net 1)
+	)
+	(via
+		(at 29.845 97.79)
+		(size 0.6)
+		(drill 0.3)
+		(layers "F.Cu" "B.Cu")
+		(free yes)
+		(net 1)
+	)
+	(via
 		(at 63.119 100.203)
 		(size 0.6)
@@
 	)
 	(via
+		(at 36.83 85.09)
+		(size 0.6)
+		(drill 0.3)
+		(layers "F.Cu" "B.Cu")
+		(free yes)
+		(net 1)
+	)
+	(via
 		(at 50.165 91.44)
 		(size 0.6)
@@
 	)
 	(via
+		(at 47.625 88.9)
+		(size 0.6)
+		(drill 0.3)
+		(layers "F.Cu" "B.Cu")
+		(free yes)
+		(net 1)
+	)
+	(via
 		(at 62.865 97.155)
 		(size 0.6)
@@
 		(net 1)
 	)
+	(via
+		(at 41.275 95.885)
+		(size 0.6)
+		(drill 0.3)
+		(layers "F.Cu" "B.Cu")
+		(net 1)
+	)
+	(via
+		(at 55.372 84.53734)
+		(size 0.6)
+		(drill 0.3)
+		(layers "F.Cu" "B.Cu")
+		(net 1)
+	)
 	(segment
 		(start 42.84 59.604)
@@
 	)
 	(segment
-		(start 57.531 85.344)
-		(end 60.383 85.344)
+		(start 49.784 77.597)
+		(end 49.911 77.597)
 		(width 0.254)
 		(layer "In2.Cu")
@@
 	)
 	(segment
-		(start 49.784 77.597)
-		(end 57.531 85.344)
+		(start 57.658 85.344)
+		(end 60.383 85.344)
 		(width 0.254)
 		(layer "In2.Cu")
@@
 	)
 	(segment
+		(start 49.911 77.597)
+		(end 57.658 85.344)
+		(width 0.254)
+		(layer "In2.Cu")
+		(net 97)
+	)
+	(segment
 		(start 52.752911 80.209105)
 		(end 52.181503 79.637697)
@@
 		(net 107)
 	)
-	(via
-		(at 46.355 94.615)
-		(size 0.6)
-		(drill 0.3)
-		(layers "F.Cu" "B.Cu")
-		(net 107)
-	)

Commit message: Finalizing Board Routing
Parts:
- removed the D4 at (70.5, 105.3)
- added J4: PWM, Connector_PinHeader_2.54mm:PinHeader_2x03_P2.54mm_Vertical, F.Cu at (50.5, 64.8)
- added R14: 10k, Resistor_SMD:R_0603_1608Metric, F.Cu at (64.6, 103.9)
- added R15: 10k, Resistor_SMD:R_0603_1608Metric, F.Cu at (66.4, 103.9)
- added R16: 10k, Resistor_SMD:R_0603_1608Metric, F.Cu at (62.9, 103.9)
- U2: value FT231XQ -> FT232RQ; footprint Package_DFN_QFN:QFN-20-1EP_4x4mm_P0.5mm_EP2.5x2.5mm -> Package_DFN_QFN:QFN-32-1EP_5x5mm_P0.5mm_EP3.1x3.1mm
- moved C15 7.01 mm to (73.0, 106.0), turned to 180 degrees
- moved L1 4.21 mm to (69.7, 105.9), turned to 180 degrees
- moved C14 2.05 mm to (57.7, 100.3)
- moved C13 1.28 mm to (62.9, 93.2), turned to -90 degrees
- moved U2 0.92 mm to (62.3, 97.9)
- moved C12 0.40 mm to (64.4, 93.2), turned to -90 degrees
- moved C16 0.25 mm to (70.2, 108.0)
- renumbered C31 to C18, C33 to C19, C32 to C20, C34 to C21, C18 to C22, C19 to C23, C20 to C24, C21 to C25, C22 to C26, C23 to C27, C24 to C28, C25 to C29, C26 to C30, C27 to C31, C28 to C32, C35 to C33, C29 to C34, C30 to C35, D5 to D4, D7 to D5, J9 to J10, J10 to J11, J4 to J5, J5 to J6, J6 to J7, J7 to J8, J8 to J9, R15 to R17, R14 to R18, R16 to R19, R17 to R20, R18 to R21, R19 to R22, R20 to R23, R21 to R24, R22 to R25, R23 to R26, R24 to R27, R25 to R28, R45 to R29, R26 to R30, R27 to R31, R28 to R32, R29 to R33, R30 to R34, R31 to R35, R32 to R36, R33 to R37, R34 to R38, R35 to R39, R36 to R40, R37 to R41, R38 to R42, R39 to R43, R40 to R44, R41 to R45, R42 to R46, R43 to R47, R44 to R48, TP4 to TP2, TP2 to TP3, TP3 to TP4
Connections:
- C14 pad 1: +3V3 -> +5V
- C15 pad 2: Net-(D4-K) -> VBUS
- D4 pad 1: RX_LED -> TX_LED
- D5 pad 1: TX_LED -> RX_LED
- L1 pad 1: Net-(D4-K) -> VBUS
- R7 pad 2: Net-(U2-USBDP) -> Net-(U2-USBD+)
- R8 pad 2: Net-(U2-USBDM) -> Net-(U2-USBD-)
- U1 pad 10: PWM2 -> PB2
- U1 pad 11: PWM3 -> PB3
- U1 pad 8: PWM0 -> PB0
- U1 pad 9: PWM1 -> PB1
- U2 pad 1: TX -> +5V
- U2 pad 10: +3V3 -> Net-(U2-CBUS2)
- U2 pad 11: +3V3 -> Net-(U2-CBUS3)
- U2 pad 12: +5V -> unconnected-(U2-NC-Pad12)
- U2 pad 13: GND -> unconnected-(U2-NC-Pad13)
- U2 pad 14: RX_LED -> Net-(U2-USBD+)
- U2 pad 15: unconnected-(U2-CBUS0-Pad15) -> Net-(U2-USBD-)
- U2 pad 16: unconnected-(U2-CBUS3-Pad16) -> +3V3
- U2 pad 17: RX -> GND
- U2 pad 18: unconnected-(U2-~{DTR}-Pad18) -> +5V
- U2 pad 19: unconnected-(U2-~{RTS}-Pad19) -> +5V
- U2 pad 2: unconnected-(U2-~{RI}-Pad2) -> TX
- U2 pad 20: +3V3 -> GND
- U2 pad 21: GND -> RX_LED
- U2 pad 3: GND -> unconnected-(U2-RI-Pad3)
- U2 pad 4: unconnected-(U2-~{DSR}-Pad4) -> GND
- U2 pad 7: TX_LED -> unconnected-(U2-DCD-Pad7)
- U2 pad 8: Net-(U2-USBDP) -> unconnected-(U2-CTS-Pad8)
- U2 pad 9: Net-(U2-USBDM) -> Net-(U2-CBUS4)
Routing:
- net PB1: track 0.00 -> 28.6 mm, vias 0 -> 1
- net PB0: track 0.00 -> 26.2 mm, vias 0 -> 1
- net PB3: track 0.00 -> 24.5 mm, vias 0 -> 1
- net PB2: track 0.00 -> 24.0 mm, vias 0 -> 1
- net +3V3: track 18.3 -> 2.32 mm, vias 2 -> 0
- net GND: track 32.1 -> 38.5 mm, vias 41 -> 52
- net ~{RESET}: track 27.5 -> 33.6 mm
- net +5V: track 69.6 -> 75.6 mm, vias 22 -> 26
- net Net-(D4-K): track 5.40 -> 0.00 mm
- net Net-(U2-CBUS3): track 0.00 -> 5.39 mm
- net Net-(U2-CBUS2): track 0.00 -> 4.85 mm
- net TX_LED: track 17.2 -> 21.5 mm
- net Net-(U2-CBUS4): track 0.00 -> 4.20 mm
- net RX: track 23.2 -> 26.3 mm
- net Net-(U2-USBDM): track 2.64 -> 0.00 mm
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Other:
- board text added: "PWM"

Commit message: Updating BOM
Parts:
- added TP8: TestPoint, TestPoint:TestPoint_Pad_D1.0mm, F.Cu at (65.4, 109.2)
- J6: value SMA-J-P-H-ST-EM1 -> 132291
- R20, R21: value 0 -> 27
- R27, R28: value 1k -> 27
- moved C16 0.38 mm to (70.2, 108.3)
Routing:
- net +5V: track 75.6 -> 78.3 mm
- net TX: track 32.7 -> 31.1 mm
- net GND: track 38.5 -> 38.2 mm, vias 52 -> 68
Other:
- board text added: "CLK"

Commit message: Minor Updates to Board
Parts:
- added REF**: OSHW-Symbol_6.7x6mm_SilkScreen, Symbol:OSHW-Symbol_6.7x6mm_SilkScreen, F.Cu at (62.4, 18.5)
- moved TP4 10.5 mm to (38.2, 77.2)
- moved R27 7.73 mm to (33.0, 71.1), turned to 0 degrees
- moved TP3 7.12 mm to (29.0, 70.6)
- moved R28 5.41 mm to (32.9, 77.3)
- moved C1 4.50 mm to (45.0, 55.2)
- moved R1 4.50 mm to (45.0, 57.1)
- moved SW1 3.45 mm to (51.6, 56.1)
- moved C30 1.91 mm to (50.2, 35.6)
- moved C31 1.91 mm to (50.2, 39.4)
- moved R47 1.91 mm to (50.2, 33.7)
- moved TP6 1.91 mm to (50.8, 31.8)
- moved TP7 1.91 mm to (50.8, 41.3)
- moved R48 1.90 mm to (50.2, 37.5)
Connections:
- TP3 pad 1: Net-(J8-In) -> Net-(U5A-+)
- TP4 pad 1: Net-(J9-In) -> Net-(U5B-+)
Routing:
- net Net-(U5A--): track 10.5 -> 3.07 mm
- net Net-(J8-In): track 6.14 -> 13.6 mm
- net Net-(U5B--): track 11.3 -> 5.13 mm
- net Net-(J9-In): track 6.14 -> 9.95 mm
- net ~{RESET}: track 33.6 -> 30.0 mm
- net Net-(U5A-+): track 5.06 -> 8.55 mm
- net Net-(U5B-+): track 4.74 -> 7.05 mm
- net GND: track 38.2 -> 36.6 mm, vias 68 -> 86
- net Net-(R1-Pad1): track 9.97 -> 9.06 mm
- net Net-(R45-Pad1): track 12.4 -> 11.5 mm
- net Net-(R44-Pad1): track 21.9 -> 21.1 mm
- net ADC_1: track 15.6 -> 14.8 mm
- net ADC_0: track 9.83 -> 10.5 mm
Other:
- board text added: "${TITLE} ${REVISION} ${COMMENT1}"
- board text added: "PB0"
- board text added: "PB1"
- board text added: "PB2"
- board text added: "PB3"
- board text added: "PD0"
- board text added: "PD1"
- board text added: "PD2"
- board text added: "PD3"
- board text added: "PE0"
- board text added: "PE1"
- board text added: "PE2"
- board text added: "PE3"
- board text added: "PE4"
- board text added: "PE5"
- board text added: "PE6"
- board text added: "PE7"
- board text added: "PG0"
- board text added: "PG1"
- board text added: "PG2"
- board text added: "PG3"
- board text added: "PG4"
- board text added: "PG5"
- board text added: "PG6"
- board text added: "PG7"
- board text removed: "${TITLE} ${COMMENT1} ${REVISION}"

Commit message: Adding gerbers
Parts:
- J6: value 132291 -> 2057-RF2-19A-T-00-50-G-ND
Changed lines of the file:
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@@
 			(outputformat 1)
 			(mirror no)
-			(drillshape 1)
+			(drillshape 0)
 			(scaleselection 1)
-			(outputdirectory "")
+			(outputdirectory "gerbers")
 		)
 	)
@@
 		(tags "resistor")
 		(property "Reference" "R27"
-			(at 0.127 -1.524 360)
+			(at 0.127 -1.524 0)
 			(layer "F.SilkS")
 			(effects
@@
 		)
 		(property "Value" "27"
-			(at 0 1.43 360)
+			(at 0 1.43 0)
 			(layer "F.Fab")
 			(effects
@@
 		)
 		(fp_text user "${REFERENCE}"
-			(at 0 0 360)
+			(at 0 0 0)
 			(layer "F.Fab")
 			(effects
@@
 			)
 		)
+		(property "Digikey" "900-0702461602-ND"
+			(at 0 0 180)
+			(unlocked yes)
+			(layer "F.Fab")
+			(hide yes)
+			(effects
+				(font
+					(size 1 1)
+					(thickness 0.15)
+				)
+			)
+		)
 		(property ki_fp_filters "Connector*:*_2x??_*")
 		(sheetname "Root")
@@
 			)
 		)
+		(property "Digikey" "900-0702461602-ND"
+			(at 0 0 180)
+			(unlocked yes)
+			(layer "F.Fab")
+			(hide yes)
+			(effects
+				(font
+					(size 1 1)
+					(thickness 0.15)
+				)
+			)
+		)
 		(property ki_fp_filters "Connector*:*_2x??_*")
 		(sheetname "Root")
@@
 			)
 		)
-		(property "Value" "132291"
+		(property "Value" "2057-RF2-19A-T-00-50-G-ND"
 			(at 0 5 -90)
 			(layer "F.Fab")
@@
 			)
 		)
-		(property "Digikey" "SAM8857-ND"
+		(property "Digikey" "2057-RF2-19A-T-00-50-G-ND"
 			(at 0 0 -90)
 			(unlocked yes)
