File: Hardware/S-Band Amplifier/S-Band Amplifier/S-Band Amplifier.kicad_pcb (KiCad board)
At the start: 2 copper layers, 70 x 40 mm, 14 parts, among them J1 Conn_Coaxial, J2 Conn_Coaxial

Commit message: Updating Amplifier board
Parts:
- added H1: 4-40, B12T_MountingHole:4-40_Hole_Pad, F.Cu at (80.0, 75.0)
- added H2: 4-40, B12T_MountingHole:4-40_Hole_Pad, F.Cu at (55.0, 105.0)
- added H3: 4-40, B12T_MountingHole:4-40_Hole_Pad, F.Cu at (105.0, 75.0)
- added H4: 4-40, B12T_MountingHole:4-40_Hole_Pad, F.Cu at (105.0, 105.0)
- added H5: 4-40, B12T_MountingHole:4-40_Hole_Pad, F.Cu at (80.0, 105.0)
- added H6: 4-40, B12T_MountingHole:4-40_Hole_Pad, F.Cu at (55.0, 75.0)
- C11: value C_Small -> 12pF
- R1: value R_Small_US -> 5.1
- moved C9 7.30 mm to (61.8, 78.3)
- moved C8 2.50 mm to (66.0, 78.5)
- moved J2 1.14 mm to (46.1, 90.0)
- moved R1 1.05 mm to (75.5, 82.6), turned to -90 degrees
- moved C1 1.00 mm to (68.5, 90.0)
- moved C4 1.00 mm to (91.5, 90.0)
- moved J1 0.91 mm to (111.9, 90.0)
- moved C6 0.83 mm to (65.7, 91.1)
- moved C2 0.78 mm to (90.3, 94.8)
- moved C3 0.76 mm to (90.3, 85.2)
- moved C5 0.44 mm to (100.6, 91.2), turned to 90 degrees
- moved C10 0.33 mm to (98.0, 80.7)
Routing:
- net GND: vias 0 -> 1152
Other:
- board text added: "${TITLE} ${REVISION} ${COMMENT1} 0.8 mm FR4"

Commit message: Finalizing Amplifier Board
Parts:
- moved C10 11.5 mm to (88.9, 73.6), turned to 180 degrees
- moved C5 4.60 mm to (96.0, 91.2)
- moved C11 3.69 mm to (98.2, 80.5)
- moved C7 1.00 mm to (70.0, 78.5)
- moved C8 1.00 mm to (65.0, 78.5)
- moved C9 0.20 mm to (62.0, 78.3)
Routing:
- net GND: vias 1152 -> 1163
Changed lines of the file:
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@@
 	(footprint "Capacitor_SMD:C_0805_2012Metric"
 		(layer "F.Cu")
-		(at 94.5 80.5 -90)
+		(at 98.19 80.45 -90)
 		(descr "Capacitor SMD 0805 (2012 Metric), square (rectangular) end terminal, IPC_7351 nominal, (Body size source: IPC-SM-782 page 76, https://www.pcb-3d.com/wordpress/wp-content/uploads/ipc-sm-782a_amendment_1_and_2.pdf, https://docs.google.com/spreadsheets/d/1BsfQQcO9C6DZCsRaXUlFlo91Tg2WpOkGARC1WS5S8t0/edit?usp=sharing), generated with kicad-footprint-generator")
 		(tags "capacitor")
@@
 	(footprint "Capacitor_SMD:C_0805_2012Metric"
 		(layer "F.Cu")
-		(at 66 78.45 90)
+		(at 65 78.45 90)
 		(descr "Capacitor SMD 0805 (2012 Metric), square (rectangular) end terminal, IPC_7351 nominal, (Body size source: IPC-SM-782 page 76, https://www.pcb-3d.com/wordpress/wp-content/uploads/ipc-sm-782a_amendment_1_and_2.pdf, https://docs.google.com/spreadsheets/d/1BsfQQcO9C6DZCsRaXUlFlo91Tg2WpOkGARC1WS5S8t0/edit?usp=sharing), generated with kicad-footprint-generator")
 		(tags "capacitor")
@@
 	(footprint "Capacitor_SMD:C_0805_2012Metric"
 		(layer "F.Cu")
-		(at 100.6 91.2 90)
+		(at 96 91.2 90)
 		(descr "Capacitor SMD 0805 (2012 Metric), square (rectangular) end terminal, IPC_7351 nominal, (Body size source: IPC-SM-782 page 76, https://www.pcb-3d.com/wordpress/wp-content/uploads/ipc-sm-782a_amendment_1_and_2.pdf, https://docs.google.com/spreadsheets/d/1BsfQQcO9C6DZCsRaXUlFlo91Tg2WpOkGARC1WS5S8t0/edit?usp=sharing), generated with kicad-footprint-generator")
 		(tags "capacitor")
@@
 	(footprint "Capacitor_SMD:C_1210_3225Metric"
 		(layer "F.Cu")
-		(at 98 80.7 -90)
+		(at 88.875 73.63 180)
 		(descr "Capacitor SMD 1210 (3225 Metric), square (rectangular) end terminal, IPC_7351 nominal, (Body size source: IPC-SM-782 page 76, https://www.pcb-3d.com/wordpress/wp-content/uploads/ipc-sm-782a_amendment_1_and_2.pdf), generated with kicad-footprint-generator")
 		(tags "capacitor")
 		(property "Reference" "C10"
-			(at 0 -2.3 90)
+			(at 0 -2.3 180)
 			(layer "F.SilkS")
 			(hide yes)
@@
 		)
 		(property "Value" "10uF"
-			(at 0 2.3 90)
+			(at 0 2.3 180)
 			(layer "F.Fab")
 			(effects
@@
 		)
 		(property "Footprint" "Capacitor_SMD:C_1210_3225Metric"
-			(at 0 0 -90)
+			(at 0 0 180)
 			(unlocked yes)
 			(layer "F.Fab")
@@
 		)
 		(property "Datasheet" ""
-			(at 0 0 -90)
+			(at 0 0 180)
 			(unlocked yes)
 			(layer "F.Fab")
@@
 		)
 		(property "Description" "Unpolarized capacitor, small symbol"
-			(at 0 0 -90)
+			(at 0 0 180)
 			(unlocked yes)
 			(layer "F.Fab")
@@
 		)
 		(fp_line
-			(start -2.3 1.6)
-			(end -2.3 -1.6)
+			(start 2.3 1.6)
+			(end -2.3 1.6)
 			(stroke
 				(width 0.05)
@@
 		)
 		(fp_line
-			(start 2.3 1.6)
-			(end -2.3 1.6)
+			(start 2.3 -1.6)
+			(end 2.3 1.6)
 			(stroke
 				(width 0.05)
@@
 		)
 		(fp_line
-			(start -2.3 -1.6)
-			(end 2.3 -1.6)
+			(start -2.3 1.6)
+			(end -2.3 -1.6)
 			(stroke
 				(width 0.05)
@@
 		)
 		(fp_line
-			(start 2.3 -1.6)
-			(end 2.3 1.6)
+			(start -2.3 -1.6)
+			(end 2.3 -1.6)
 			(stroke
 				(width 0.05)
@@
 		)
 		(fp_line
-			(start -1.6 1.25)
-			(end -1.6 -1.25)
+			(start 1.6 1.25)
+			(end -1.6 1.25)
 			(stroke
 				(width 0.1)
@@
 		)
 		(fp_line
-			(start 1.6 1.25)
-			(end -1.6 1.25)
+			(start 1.6 -1.25)
+			(end 1.6 1.25)
 			(stroke
 				(width 0.1)
@@
 		)
 		(fp_line
-			(start -1.6 -1.25)
-			(end 1.6 -1.25)
+			(start -1.6 1.25)
+			(end -1.6 -1.25)
 			(stroke
 				(width 0.1)
@@
 		)
 		(fp_line
-			(start 1.6 -1.25)
-			(end 1.6 1.25)
+			(start -1.6 -1.25)
+			(end 1.6 -1.25)
 			(stroke
 				(width 0.1)
@@
 		)
 		(fp_text user "${REFERENCE}"
-			(at 0 0 90)
+			(at 0 0 180)
 			(layer "F.Fab")
 			(effects
@@
 		)
 		(pad "1" smd roundrect
-			(at -1.475 0 270)
+			(at -1.475 0 180)
 			(size 1.15 2.7)
 			(layers "F.Cu" "F.Paste" "F.Mask")
@@
 		)
 		(pad "2" smd roundrect
-			(at 1.475 0 270)
+			(at 1.475 0 180)
 			(size 1.15 2.7)
 			(layers "F.Cu" "F.Paste" "F.Mask")
@@
 	(footprint "Capacitor_SMD:C_0805_2012Metric"
 		(layer "F.Cu")
-		(at 69 78.45 90)
+		(at 70 78.45 90)
 		(descr "Capacitor SMD 0805 (2012 Metric), square (rectangular) end terminal, IPC_7351 nominal, (Body size source: IPC-SM-782 page 76, https://www.pcb-3d.com/wordpress/wp-content/uploads/ipc-sm-782a_amendment_1_and_2.pdf, https://docs.google.com/spreadsheets/d/1BsfQQcO9C6DZCsRaXUlFlo91Tg2WpOkGARC1WS5S8t0/edit?usp=sharing), generated with kicad-footprint-generator")
 		(tags "capacitor")
@@
 	(footprint "Capacitor_SMD:C_1210_3225Metric"
 		(layer "F.Cu")
-		(at 61.8 78.3 90)
+		(at 62 78.3 90)
 		(descr "Capacitor SMD 1210 (3225 Metric), square (rectangular) end terminal, IPC_7351 nominal, (Body size source: IPC-SM-782 page 76, https://www.pcb-3d.com/wordpress/wp-content/uploads/ipc-sm-782a_amendment_1_and_2.pdf), generated with kicad-footprint-generator")
 		(tags "capacitor")
@@
 	(gr_poly
 		(pts
-			(xy 83.965 86) (xy 83.965 80) (xy 85.465 78.5) (xy 98.965 78.5) (xy 98.965 75) (xy 88.965 75) (xy 88.965 70.5)
+			(xy 83.965 86) (xy 83.965 80) (xy 85.465 78.5) (xy 98.965 78.5) (xy 98.965 75) (xy 89.765 75) (xy 89.765 70.5)
 			(xy 96.965 70.5) (xy 96.965 73.5) (xy 98.9 73.5) (xy 100.465 75.1) (xy 100.465 78.3) (xy 98.8 80)
 			(xy 85.465 80) (xy 85.465 86)
@@
 		(layer "Cmts.User")
 		(pts
-			(xy 45 110) (xy 115 110)
+			(xy 55 75) (xy 80 75)
+		)
+		(height -8)
+		(gr_text "25.0000 mm"
+			(at 67.5 65.85 0)
+			(layer "Cmts.User")
+			(effects
+				(font
+					(size 1 1)
+					(thickness 0.15)
+				)
+			)
+		)
+		(format
+			(prefix "")
+			(suffix "")
+			(units 3)
+			(units_format 1)
+			(precision 4)
+		)
+		(style
+			(thickness 0.1)
+			(arrow_length 1.27)
+			(text_position_mode 0)
+			(extension_height 0.58642)
+			(extension_offset 0.5) keep_text_aligned)
+	)
+	(dimension
+		(type aligned)
+		(layer "Cmts.User")
+		(pts
+			(xy 91.815 90) (xy 96 90)
+		)
+		(height -2.5)
+		(gr_text "4.1850 mm"
+			(at 93.9075 86.35 0)
+			(layer "Cmts.User")
+			(effects
+				(font
+					(size 1 1)
+					(thickness 0.15)
+				)
+			)
+		)
+		(format
+			(prefix "")
+			(suffix "")
+			(units 3)
+			(units_format 1)
+			(precision 4)
+		)
+		(style
+			(thickness 0.1)
+			(arrow_length 1.27)
+			(text_position_mode 0)
+			(extension_height 0.58642)
+			(extension_offset 0.5) keep_text_aligned)
+	)
+	(dimension
+		(type aligned)
+		(layer "Cmts.User")
+		(pts
+			(xy 55 75) (xy 55 105)
+		)
+		(height 25)
+		(gr_text "30.0000 mm"
+			(at 28.85 90 90)
+			(layer "Cmts.User")
+			(effects
+				(font
+					(size 1 1)
+					(thickness 0.15)
+				)
+			)
+		)
+		(format
+			(prefix "")
+			(suffix "")
+			(units 3)
+			(units_format 1)
+			(precision 4)
+		)
+		(style
+			(thickness 0.1)
+			(arrow_length 1.27)
+			(text_position_mode 0)
+			(extension_height 0.58642)
+			(extension_offset 0.5) keep_text_aligned)
+	)
+	(dimension
+		(type aligned)
+		(layer "Cmts.User")
+		(pts
+			(xy 44 110) (xy 114 110)
 		)
 		(height 2.7)
 		(gr_text "70.0000 mm"
-			(at 80 111.55 0)
+			(at 79 111.55 0)
+			(layer "Cmts.User")
+			(effects
+				(font
+					(size 1 1)
+					(thickness 0.15)
+				)
+			)
+		)
+		(format
+			(prefix "")
+			(suffix "")
+			(units 3)
+			(units_format 1)
+			(precision 4)
+		)
+		(style
+			(thickness 0.1)
+			(arrow_length 1.27)
+			(text_position_mode 0)
+			(extension_height 0.58642)
+			(extension_offset 0.5) keep_text_aligned)
+	)
+	(dimension
+		(type aligned)
+		(layer "Cmts.User")
+		(pts
+			(xy 55 75) (xy 105 75)
+		)
+		(height -13)
+		(gr_text "50.0000 mm"
+			(at 80 60.85 0)
 			(layer "Cmts.User")
 			(effects
@@
 	)
 	(via
+		(at 55 93)
+		(size 0.6)
+		(drill 0.3)
+		(layers "F.Cu" "B.Cu")
+		(net 4)
+	)
+	(via
 		(at 103 99)
 		(size 0.6)
@@
 	)
 	(via
+		(at 59 93)
+		(size 0.6)
+		(drill 0.3)
+		(layers "F.Cu" "B.Cu")
+		(net 4)
+	)
+	(via
 		(at 80.5 86.15)
 		(size 0.6)
@@
 	)
 	(via
+		(at 51 93)
+		(size 0.6)
+		(drill 0.3)
+		(layers "F.Cu" "B.Cu")
+		(net 4)
+	)
+	(via
 		(at 80.85 90.05)
 		(size 0.6)
@@
 	)
 	(via
+		(at 45 93)
+		(size 0.6)
+		(drill 0.3)
+		(layers "F.Cu" "B.Cu")
+		(net 4)
+	)
+	(via
 		(at 78.05 85.6)
 		(size 0.6)
@@
 	)
 	(via
+		(at 65 93)
+		(size 0.6)
+		(drill 0.3)
+		(layers "F.Cu" "B.Cu")
+		(net 4)
+	)
+	(via
 		(at 103 81)
 		(size 0.6)
@@
 	)
 	(via
+		(at 57 93)
+		(size 0.6)
+		(drill 0.3)
+		(layers "F.Cu" "B.Cu")
+		(net 4)
+	)
+	(via
 		(at 77 107)
 		(size 0.6)
@@
 	)
 	(via
+		(at 58 108)
+		(size 0.6)
+		(drill 0.3)
+		(layers "F.Cu" "B.Cu")
+		(net 4)
+	)
+	(via
 		(at 80.5 83.55)
 		(size 0.6)
@@
 	)
 	(via
+		(at 61 93)
+		(size 0.6)
+		(drill 0.3)
+		(layers "F.Cu" "B.Cu")
+		(net 4)
+	)
+	(via
 		(at 108 100)
 		(size 0.6)
@@
 	)
 	(via
-		(at 77.4 94.8)
-		(size 0.6)
-		(drill 0.3)
-		(layers "F.Cu" "B.Cu")
-		(free yes)
-		(net 4)
-	)
-	(via
 		(at 109.7 92.15)
 		(size 0.6)
@@
 	)
 	(via
+		(at 53 93)
+		(size 0.6)
+		(drill 0.3)
+		(layers "F.Cu" "B.Cu")
+		(net 4)
+	)
+	(via
 		(at 55.25 91.95)
 		(size 0.6)
@@
 	)
 	(via
+		(at 49 93)
+		(size 0.6)
+		(drill 0.3)
+		(layers "F.Cu" "B.Cu")
+		(net 4)
+	)
+	(via
 		(at 74.15 75.6)
 		(size 0.6)
@@
 	)
 	(via
+		(at 47 93)
+		(size 0.6)
+		(drill 0.3)
+		(layers "F.Cu" "B.Cu")
+		(net 4)
+	)
+	(via
 		(at 52 94)
 		(size 0.6)
@@
 		(net 4)
 	)
+	(via
+		(at 63 93)
+		(size 0.6)
+		(drill 0.3)
+		(layers "F.Cu" "B.Cu")
+		(net 4)
+	)
