File: Hardware/S-Band Amplifier/S-Band Amplifier/S-Band Amplifier.kicad_sch (KiCad schematic)
At the start: 16 parts, among them J1 Conn_Coaxial, J2 Conn_Coaxial, Q1 BLP9G0722-20G

Commit message: Updating Amplifier board
Parts:
- added H1, H2, H3, H4, H5, H6: 4-40, B12T_MountingHole:4-40_Hole_Pad, symbol Mechanical:MountingHole_Pad
Connections:
- net GND: now also H1.1, H2.1, H3.1, H4.1, H5.1, H6.1

Commit message: Finalizing Amplifier Board
Parts:
- removed C8: 12pF, Capacitor_SMD:C_0805_2012Metric, symbol Device:C_Small
- C1: value 5.6pF -> 12pF
- C3: now not fitted
- C7: value 62pF -> 68pF
Other:
- moved on the sheet: C9
