File: Hardware/GaN Gate Driver/GaN Gate Driver.kicad_pcb (KiCad board)
At the start: 2 copper layers, 38.1 x 38.1 mm, 33 parts, among them J1 SMA-J-P-X-ST-EM1, J2 Conn_01x03_Socket, J3 Conn_01x02_Socket, U1 LT1804

Commit message: Adding gerbers
Routing:
- net GND: vias 12 -> 45
