File: Hardware/X-Band Amplifier QPA2598/X-Band Amplifier QPA2598.kicad_pcb (KiCad board)
At the start: 4 copper layers, 25.4 x 25.4 mm, 17 parts, among them J1 901-10513-3, J2 901-10513-3, U1 QPA2598

Commit message: Adding Gerber files
Routing:
- net VD: track 7.88 -> 7.25 mm
- net GND: vias 202 -> 209
Changed lines of the file:
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@@
 	)
 	(gr_text "GND"
-		(at 134.7216 54.3052 0)
+		(at 134.493 54.3052 0)
 		(layer "F.SilkS")
 		(effects
@@
 	)
 	(via
-		(at 144.399 60.96)
+		(at 144.653 60.96)
 		(size 0.6)
 		(drill 0.3)
@@
 	)
 	(via
+		(at 141.351 60.96)
+		(size 0.6)
+		(drill 0.3)
+		(layers "F.Cu" "B.Cu")
+		(free yes)
+		(net 1)
+	)
+	(via
 		(at 135.763 62.484)
 		(size 0.6)
@@
 	(via
 		(at 150.241 65.151)
+		(size 0.6)
+		(drill 0.3)
+		(layers "F.Cu" "B.Cu")
+		(free yes)
+		(net 1)
+	)
+	(via
+		(at 136.906 60.579)
 		(size 0.6)
 		(drill 0.3)
@@
 	)
 	(via
+		(at 133.35 60.96)
+		(size 0.6)
+		(drill 0.3)
+		(layers "F.Cu" "B.Cu")
+		(free yes)
+		(net 1)
+	)
+	(via
 		(at 140.2 62.5)
 		(size 0.5)
@@
 	)
 	(via
+		(at 141.986 60.96)
+		(size 0.6)
+		(drill 0.3)
+		(layers "F.Cu" "B.Cu")
+		(free yes)
+		(net 1)
+	)
+	(via
 		(at 132.207 65.151)
 		(size 0.6)
@@
 	)
 	(via
+		(at 142.748 60.96)
+		(size 0.6)
+		(drill 0.3)
+		(layers "F.Cu" "B.Cu")
+		(free yes)
+		(net 1)
+	)
+	(via
 		(at 151.511 61.849)
 		(size 0.6)
@@
 	)
 	(via
-		(at 142.621 65.913)
+		(at 142.748 66.04)
 		(size 0.6)
 		(drill 0.3)
@@
 	)
 	(via
-		(at 145.542 60.96)
+		(at 145.669 60.96)
 		(size 0.6)
 		(drill 0.3)
@@
 	)
 	(via
+		(at 139.446 55.245)
+		(size 0.6)
+		(drill 0.3)
+		(layers "F.Cu" "B.Cu")
+		(free yes)
+		(net 1)
+	)
+	(via
 		(at 147.066 65.151)
 		(size 0.6)
@@
 	)
 	(via
-		(at 143.256 60.96)
+		(at 143.637 60.96)
 		(size 0.6)
 		(drill 0.3)
@@
 	)
 	(via
-		(at 134.112 60.325)
+		(at 134.239 60.071)
 		(size 0.6)
 		(drill 0.3)
@@
 	)
 	(via
+		(at 134.874 60.96)
+		(size 0.6)
+		(drill 0.3)
+		(layers "F.Cu" "B.Cu")
+		(free yes)
+		(net 1)
+	)
+	(via
 		(at 136.779 69.215)
 		(size 0.6)
@@
 	)
 	(segment
-		(start 141.2342 55.245)
-		(end 142.367 55.245)
-		(width 1.27)
-		(layer "F.Cu")
-		(net 4)
-	)
-	(segment
 		(start 140.2 60.335)
 		(end 140.21 60.325)
 		(width 0.25)
+		(layer "F.Cu")
+		(net 4)
+	)
+	(segment
+		(start 140.396 57.785)
+		(end 140.396 57.1652)
+		(width 1.27)
 		(layer "F.Cu")
 		(net 4)
@@
 	)
 	(segment
-		(start 140.396 57.785)
-		(end 140.396 56.0832)
+		(start 142.3162 55.245)
+		(end 142.367 55.245)
+		(width 1.27)
+		(layer "F.Cu")
+		(net 4)
+	)
+	(segment
+		(start 140.396 57.1652)
+		(end 142.3162 55.245)
 		(width 1.27)
 		(layer "F.Cu")
@@
 		(end 140.206 57.975)
 		(width 0.4)
-		(layer "F.Cu")
-		(net 4)
-	)
-	(segment
-		(start 140.396 56.0832)
-		(end 141.2342 55.245)
-		(width 1.27)
 		(layer "F.Cu")
 		(net 4)
@@
 		(polygon
 			(pts
-				(xy 141.097 70.866) (xy 143.637 70.866) (xy 143.637 75.946) (xy 141.097 75.946)
+				(xy 140.957 70.866) (xy 143.497 70.866) (xy 143.497 75.946) (xy 140.957 75.946)
 			)
 		)
