File: Hardware/GaN Drain Driver/GaN Drain Driver.kicad_pcb (KiCad board)
At the start: 2 copper layers, 88.9 x 38.1 mm, 70 parts, among them J1 SMA-J-P-H-ST-EM1, J2 Conn_01x02_Socket, J3 Conn_01x02_Socket, J4 Conn_01x02_Socket, Q1 NVD360N65S3T4G, Q2 NVD360N65S3T4G, U1 LM317_SOT-223, U2 IRS2008S, U3 LM317_SOT-223, U5 LT1804, U6 LM393, U7 R1SE

Commit message: Updating schematic
Parts:
- removed R16: 10k, Resistor_SMD:R_0805_2012Metric
- added C24: 10uF, Capacitor_SMD:C_0805_2012Metric, F.Cu at (193.4, 50.5)
- added R18: 10k, Resistor_SMD:R_0805_2012Metric, F.Cu at (193.4, 53.4)
- added R19: 10k, Resistor_SMD:R_0805_2012Metric, F.Cu at (193.4, 56.4)
- D6: value D_Zener -> 3.3V
- R17: value 10k -> 100k
- moved J4 89.8 mm to (66.2, 60.3), turned to 90 degrees
- moved R3 4.10 mm to (107.8, 50.0)
- moved C5 4.10 mm to (107.8, 47.5)
- moved C6 4.10 mm to (119.3, 49.4)
- moved D3 4.10 mm to (113.6, 46.5)
- moved R4 4.10 mm to (107.8, 52.6)
- moved R5 4.10 mm to (119.3, 55.1)
- moved R6 4.10 mm to (119.3, 52.6)
- moved U2 4.10 mm to (113.5, 50.9)
- turned D2 to 180 degrees
Connections:
- R14 pad 1: Net-(R14-Pad1) -> COMP_OUT
- R17 pad 1: GND -> +3.3V REF
- U6 pad 1: Net-(R14-Pad1) -> COMP_OUT
- U6 pad 7: unconnected-(U6-Pad7) -> COMP_OUT

Commit message: working on board layout
Parts:
- removed C4: 10uF, Capacitor_SMD:C_0805_2012Metric
- removed the C7 at (83.2, 30.7)
- added TP7: TestPoint, TestPoint:TestPoint_Pad_D1.0mm, F.Cu at (67.9, 46.3)
- J2: footprint Connector_PinSocket_2.54mm:PinSocket_1x02_P2.54mm_Vertical -> Connector_Molex:Molex_KK-254_AE-6410-02A_1x02_P2.54mm_Vertical
- J3: renamed from J4; footprint Connector_PinSocket_2.54mm:PinSocket_1x02_P2.54mm_Vertical -> Connector_Molex:Molex_KK-254_AE-6410-02A_1x02_P2.54mm_Vertical
- J4: renamed from J3; footprint Connector_PinSocket_2.54mm:PinSocket_1x02_P2.54mm_Vertical -> Connector_Molex:Molex_KK-254_AE-6410-02A_1x02_P2.54mm_Vertical
- RV1, RV2: footprint Resistor_SMD:R_0805_2012Metric -> Potentiometer_THT:Potentiometer_Bourns_3296W_Vertical
- moved R10 137.4 mm to (65.4, 103.3)
- moved R11 137.4 mm to (65.4, 106.2)
- moved D5 130.9 mm to (56.1, 52.6), turned to -90 degrees
- moved C14 125.5 mm to (78.3, 100.4)
- moved R9 124.6 mm to (65.4, 100.3)
- moved R18 123.4 mm to (65.4, 115.1)
- moved R16 122.0 mm to (65.4, 109.2)
- moved TP6 121.4 mm to (80.3, 110.0)
- moved TP5 121.4 mm to (80.3, 107.0)
- moved D4 117.9 mm to (69.8, 52.3), turned to 90 degrees
- moved TP2 117.4 mm to (64.9, 46.4)
- moved RV2 116.6 mm to (75.7, 108.7)
- moved R7 108.9 mm to (60.1, 58.3), turned to 180 degrees
- moved C17 108.9 mm to (78.3, 103.4)
- moved C22 108.8 mm to (88.5, 108.6)
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- renumbered C18 to C1, C15 to C10, C16 to C13, C24 to C14, C19 to C15, C20 to C16, C23 to C17, C13 to C18, C14 to C19, C1 to C2, C8 to C21, C21 to C22, C22 to C23, C9 to C24, C2 to C3, C17 to C6, C3 to C7, C6 to C8, C10 to C9, R3 to R1, R18 to R10, R19 to R11, R10 to R12, R11 to R13, R12 to R14, R13 to R15, R14 to R16, R4 to R17, R15 to R18, R1 to R2, R2 to R3, R5 to R4, R6 to R5, R7 to R6, R8 to R7, R9 to R8, R17 to R9, U7 to U2, U2 to U3, U3 to U4
Other:
- board size 88.9 x 38.1 mm -> 101.6 x 50.8 mm
- board text removed: "+15V"

Commit message: Working on Board Layout
Parts:
- added C20: 1000uF, Capacitor_THT:CP_Radial_D13.0mm_P5.00mm, F.Cu at (137.8, 44.5)
- added C4: 1000uF, Capacitor_THT:CP_Radial_D13.0mm_P5.00mm, F.Cu at (123.8, 44.5)
- R18: value 10k -> 10M
- moved R11 82.2 mm to (112.4, 38.7), turned to 180 degrees
- moved R16 78.3 mm to (99.7, 38.7), turned to 180 degrees
- moved R10 77.8 mm to (112.4, 41.3)
- moved C22 76.2 mm to (112.4, 36.2)
- moved R18 74.4 mm to (78.7, 41.9), turned to 180 degrees
- moved R9 73.5 mm to (112.4, 43.8), turned to 180 degrees
- moved R17 69.0 mm to (78.7, 44.5), turned to 0 degrees
- moved C23 68.7 mm to (99.7, 43.8), turned to 180 degrees
- moved TP5 67.3 mm to (106.2, 44.8)
- moved C17 65.7 mm to (99.7, 41.3)
- moved U6 65.1 mm to (106.0, 40.6)
- moved C14 63.9 mm to (112.4, 46.4)
- moved TP3 63.2 mm to (86.4, 66.7)
- moved TP6 63.0 mm to (80.0, 47.0)
- moved RV2 59.7 mm to (99.7, 54.0)
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Connections:
- R9 pad 1: +3.3V REF -> +5V
Routing:
- net +5V: track 0.00 -> 175.2 mm, vias 0 -> 6
- net Vd: track 0.00 -> 80.1 mm
- net -5V: track 0.00 -> 77.2 mm, vias 0 -> 3
- net Vg: track 0.00 -> 73.6 mm, vias 0 -> 2
- net +15V: track 0.00 -> 68.0 mm
- net +3.3V REF: track 0.00 -> 57.6 mm, vias 0 -> 3
- net Net-(Q1-G): track 0.00 -> 54.6 mm
- net -3.3V REF: track 0.00 -> 47.7 mm, vias 0 -> 1
- net Net-(Q2-G): track 0.00 -> 38.7 mm
- net ~{SD}: track 0.00 -> 29.8 mm, vias 0 -> 2
- net Net-(U5A-+): track 0.00 -> 23.2 mm
- net Net-(U6A-+): track 0.00 -> 21.8 mm, vias 0 -> 1
- net Net-(J1-In): track 0.00 -> 19.7 mm
- net Net-(R14-Pad2): track 0.00 -> 13.4 mm
- net Net-(D5-A): track 0.00 -> 12.5 mm
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- added copper zone on In1.Cu, net GND
- added copper zone on In2.Cu, net VCC
- removed copper zone on F.Cu, net Vd
Other:
- outline, holes or cut-outs redrawn
- copper layers 2 -> 4
- board text added: "Vd"
- board text added: "Vg"
- board text removed: "AMP DRAIN"

Commit message: Updating board
Parts:
- added TP8: TestPoint, TestPoint:TestPoint_Pad_D1.0mm, F.Cu at (122.1, 73.5)
- added TP9: TestPoint, TestPoint:TestPoint_Pad_D1.0mm, F.Cu at (103.2, 71.2)
- moved TP5 13.5 mm to (93.6, 49.7)
- moved J1 0.33 mm to (84.0, 27.5)
Connections:
- RV1 pad 1: +5V -> +3.3V REF
- RV1 pad 3: -5V -> -3.3V REF
Routing:
- net -5V: track 77.2 -> 91.5 mm
- net +3.3V REF: track 57.6 -> 70.4 mm
- net -3.3V REF: track 47.7 -> 60.2 mm
- net +5V: track 175.2 -> 169.5 mm, vias 6 -> 7
- net Net-(U6A-+): track 21.8 -> 26.7 mm
- net Net-(U5A-+): track 23.2 -> 25.7 mm
- net Vd: track 80.1 -> 80.5 mm, vias 0 -> 72
- net VCC: vias 1 -> 73
- net GND: vias 9 -> 10
Other:
- board text added: "+15V"
- board text added: "+3.3V REF"
- board text added: "+5V"
- board text added: "-3.3V REF"
- board text added: "-5V"
- board text added: "Vg Limit Set"
- board text added: "Vg Max"
- board text added: "Vg Set"
- board text added: "~{SD}"

Commit message: Adding gerber files
Routing:
- net GND: vias 10 -> 82

Commit message: Fixing issue with reference
Parts:
- removed D6: 3.3V, Diode_SMD:D_SOD-123
- removed the R12 at (86.4, 61.6)
- added C13: 10uF, Capacitor_SMD:C_0805_2012Metric, F.Cu at (82.5, 66.7)
- added C15: 100nF, Capacitor_SMD:C_0805_2012Metric, F.Cu at (82.5, 64.1)
- added C17: 100nF, Capacitor_SMD:C_0805_2012Metric, F.Cu at (94.6, 67.3)
- added U6: MAX6241, Package_SO:SOIC-8_3.9x4.9mm_P1.27mm, F.Cu at (88.4, 64.8)
- moved TP6 9.22 mm to (93.6, 61.0)
- moved TP8 8.78 mm to (92.7, 58.4)
- moved C16 8.28 mm to (94.6, 64.8)
- renumbered C11 to C10, C12 to C11, C13 to C12, C15 to C16, C16 to C18, C17 to C19, C18 to C21, C19 to C22, C4 to C23, C21 to C24, C22 to C25, C23 to C26, C24 to C27, C5 to C4, C6 to C5, C7 to C6, C8 to C7, C9 to C8, C10 to C9, R13 to R12, R14 to R13, R15 to R14, R16 to R15, R17 to R16, R18 to R17, TP7 to TP2, TP9 to TP3, TP2 to TP4, TP8 to TP5, TP3 to TP6, TP4 to TP7, TP5 to TP8, TP6 to TP9, U6 to U7
Connections:
- net +3.3V REF renamed +4.096V REF
- net -3.3V REF renamed -4.096V REF
Routing:
- net +5V: track 169.5 -> 137.4 mm, vias 7 -> 5
- net +4.096V REF: track 70.4 -> 47.9 mm, vias 3 -> 1
- net +15V: track 68.0 -> 78.6 mm
- net Net-(U6-NR): track 0.00 -> 2.94 mm
- net Vg: track 73.6 -> 73.1 mm
- net Net-(U7A-+): track 26.7 -> 27.2 mm
- net -4.096V REF: track 60.2 -> 60.7 mm
- net GND: vias 82 -> 93
Other:
- board text added: "+4.096V REF"
- board text removed: "+3.3V REF"

Commit message: Updating drain driver
Parts:
- removed the C11 at (55.2, 55.9)
- removed the C2 at (78.7, 64.1)
- removed the C3 at (70.5, 60.3)
- removed the C8 at (63.5, 64.1)
- removed the D1 at (80.6, 57.8)
- removed D2, D5: 1N5819HW-7-F, Diode_SMD:D_SOD-123
- removed the R2 at (74.9, 64.1)
- removed the R3 at (71.1, 64.1)
- removed the R6 at (59.7, 64.1)
- removed the R7 at (55.9, 64.1)
- removed the TP1 at (80.6, 54.0)
- removed the TP4 at (66.0, 54.0)
- removed the U1 at (75.6, 57.8)
- removed the U4 at (60.3, 57.8)
- added C13: 10uF, Capacitor_SMD:C_0805_2012Metric, F.Cu at (71.7, 52.7)
- added C7: 10uF, Capacitor_SMD:C_0805_2012Metric, F.Cu at (71.7, 63.5)
- added D3: 1N5819HW-7-F, Diode_SMD:D_SOD-123, F.Cu at (75.6, 66.4)
- added TP3: TestPoint, TestPoint:TestPoint_Pad_D1.0mm, F.Cu at (75.6, 62.6)
- added TP5: TestPoint, TestPoint:TestPoint_Pad_D1.0mm, F.Cu at (75.7, 51.8)
- added U3: L7815, Package_TO_SOT_SMD:TO-252-2, F.Cu at (63.7, 65.3)
- added U5: L7805, Package_TO_SOT_SMD:TO-252-2, F.Cu at (63.7, 54.5)
- C6: value 10uF -> 100nF
- R7: renamed from R15; value 10k -> 0
- moved C10 16.9 mm to (71.7, 56.3)
- moved C6 11.3 mm to (71.7, 67.1), turned to 90 degrees
- moved D4 9.88 mm to (75.7, 55.7)
- renumbered C4 to C1, C23 to C11, C24 to C12, C27 to C14, C25 to C15, C26 to C16, C16 to C17, C13 to C18, C9 to C19, C14 to C2, C15 to C20, C17 to C21, C18 to C22, C12 to C23, C21 to C24, C22 to C25, C19 to C3, C7 to C4, C1 to C5, C5 to C8, C20 to C9, D3 to D1, J4 to J3, J3 to J4, R12 to R10, R13 to R11, R14 to R12, R8 to R13, R9 to R2, R10 to R3, R11 to R4, R4 to R5, R5 to R6, R16 to R8, R17 to R9, RV2 to RV1, RV1 to RV2, TP8 to TP1, TP9 to TP2, TP2 to TP4, TP3 to TP7, TP7 to TP8, TP5 to TP9, U3 to U1, U7 to U2, U2 to U4, U5 to U7
Connections:
- C10 pad 1: Net-(D5-A) -> +15V
- C6 pad 1: +15V -> VCC
Routing:
- net +5V: track 137.4 -> 120.3 mm
- net +15V: track 78.6 -> 62.8 mm
- net Net-(D5-A): track 12.5 -> 0.00 mm
- net Net-(D2-A): track 12.5 -> 0.00 mm
- net VCC: track 8.54 -> 9.72 mm, vias 73 -> 80
- net Net-(U7A-+): track 25.7 -> 24.9 mm
- net GND: vias 93 -> 75

Commit message: Updating Drain Driver
Parts:
- removed the C18 at (82.5, 66.7)
- removed D3, D4: 1N5819HW-7-F, Diode_SMD:D_SOD-123
- removed the R7 at (99.7, 38.7)
- removed the R9 at (78.7, 41.9)
- R2: value 100k -> 10k
- RV1, RV2: value 10k -> 100k
- U6: value MAX6241 -> REF5040
- U7: value LT1804 -> TLV9302
- moved TP6 11.3 mm to (88.3, 70.9)
- moved TP1 5.85 mm to (88.9, 54.0)
- moved C19 1.90 mm to (80.7, 64.1)
- moved C17 1.85 mm to (92.8, 65.3)
- moved C20 1.80 mm to (92.8, 67.6)
- moved U6 1.78 mm to (86.6, 64.8)
- moved C5 1.14 mm to (62.7, 45.7)
- moved TP2 1.14 mm to (80.0, 48.1)
- renumbered C19 to C18, C20 to C19, C21 to C20, C22 to C21, C23 to C22, C24 to C23, C25 to C24, R11 to R10, R12 to R11, R13 to R12, R8 to R7, R10 to R9
Connections:
- R7 pad 2: ~{SD} -> COMP_OUT
- TP2 pad 1: ~{SD} -> COMP_OUT
- U1 pad 3: ~{SD} -> COMP_OUT
- U6 pad 3: Net-(U6-NR) -> unconnected-(U6-NR-Pad3)
Routing:
- net COMP_OUT: track 8.44 -> 41.2 mm, vias 0 -> 2
- net ~{SD}: track 29.8 -> 0.00 mm, vias 2 -> 0
- net +5V: track 120.3 -> 114.0 mm
- net Net-(U2A-+): track 27.2 -> 33.2 mm
- net +4.096V REF: track 47.9 -> 53.6 mm
- net +15V: track 62.8 -> 58.7 mm
- net VCC: track 9.72 -> 5.82 mm
- net Net-(U6-NR): track 2.94 -> 0.00 mm
- net GND: vias 75 -> 74
Other:
- board text added: "+4.1V REF"
- board text added: "-4.1V REF"
- board text removed: "+4.096V REF"
- board text removed: "-3.3V REF"
