File: Hardware/GaN Drain Driver/Power_Management.kicad_sch (KiCad schematic)
At the start: 43 parts, among them J3 Conn_01x02_Socket, J4 Conn_01x02_Socket, U2 LM393, U3 L7815, U4 R1SE, U5 L7805, U6 MAX6241, U7 LT1804

Commit message: Updating Drain Driver, Consolidating BOM
Parts:
- removed C18: 10uF, Capacitor_SMD:C_0805_2012Metric, symbol Device:C_Small
- removed D3, D4: 1N5819HW-7-F, Diode_SMD:D_SOD-123, symbol Device:D_Small

Commit message: Updating Drain Driver
Parts:
- C10, C15, C16, C17, C6: Digikey (none) -> 478-KGM21NR71H104KTCT-ND; MPN (none) -> KGM21NR71H104KT; Manufacturer (none) -> KYOCERA AVX
- C11, C12, C14: MPN (none) -> UCY2C101MHD1TO; Manufacturer (none) -> Nichicon; now not fitted
- C13, C5, C7, C8: Digikey (none) -> 1276-2891-1-ND; MPN (none) -> CL21A106KAYNNNE; Manufacturer (none) -> Samsung Electro-Mechanics
- C18: renamed from C19; Digikey (none) -> 478-KGM21NR71H104KTCT-ND; MPN (none) -> KGM21NR71H104KT; Manufacturer (none) -> KYOCERA AVX
- C19: renamed from C20; Digikey (none) -> 478-KGM21NR71H104KTCT-ND; MPN (none) -> KGM21NR71H104KT; Manufacturer (none) -> KYOCERA AVX
- C20: renamed from C21; Digikey (none) -> 478-KGM21NR71H104KTCT-ND; MPN (none) -> KGM21NR71H104KT; Manufacturer (none) -> KYOCERA AVX
- C21: renamed from C22; Digikey (none) -> 478-KGM21NR71H104KTCT-ND; MPN (none) -> KGM21NR71H104KT; Manufacturer (none) -> KYOCERA AVX
- C22: renamed from C23; Digikey (none) -> 478-KGM21NR71H104KTCT-ND; MPN (none) -> KGM21NR71H104KT; Manufacturer (none) -> KYOCERA AVX
- C23: renamed from C24; Digikey (none) -> 478-KGM21NR71H104KTCT-ND; MPN (none) -> KGM21NR71H104KT; Manufacturer (none) -> KYOCERA AVX
- C24: renamed from C25; Digikey (none) -> 478-KGM21NR71H104KTCT-ND; MPN (none) -> KGM21NR71H104KT; Manufacturer (none) -> KYOCERA AVX
- C9: MPN (none) -> UCY2C101MHD1TO; Manufacturer (none) -> Nichicon
- J3, J4: MPN (none) -> 0022272021; Manufacturer (none) -> Molex
- R10: renamed from R11; Digikey (none) -> 541-3976-1-ND; MPN (none) -> CRCW080510K0FKEAC; Manufacturer (none) -> Vishay Dale
- R11: renamed from R12; Digikey (none) -> 311-33.0CRCT-ND; MPN (none) -> RC0805FR-0733RL; Manufacturer (none) -> YAGEO
- R12: renamed from R13; Digikey (none) -> 311-33.0CRCT-ND; MPN (none) -> RC0805FR-0733RL; Manufacturer (none) -> YAGEO
- R9: renamed from R10; Digikey (none) -> 541-3976-1-ND; MPN (none) -> CRCW080510K0FKEAC; Manufacturer (none) -> Vishay Dale
- RV2: value 10k -> 100k; Digikey 3296W-103LF-ND -> 118-PV36W104C01B00-ND; MPN (none) -> PV36W104C01B00; Manufacturer (none) -> Bourns Inc.
- TP4: now left out of the parts list
- U2: MPN (none) -> LM393DT; Manufacturer (none) -> STMicroelectronics
- U3: Digikey (none) -> MC78M15CDTGOS-ND; MPN (none) -> MC78M15CDTG; Manufacturer (none) -> onsemi
- U4: MPN (none) -> R1SE-0505-R; Manufacturer (none) -> Recom Power
- U5: Digikey (none) -> MC7805BDTRKGOSCT-ND; MPN (none) -> MC7805BDTRKG; Manufacturer (none) -> onsemi
- U6: value MAX6241 -> REF5040; Digikey 175-MAX6241BESA+TCT-ND -> 296-46190-1-ND; MPN (none) -> REF5040AIDR; Manufacturer (none) -> Texas Instruments
- U7: value LT1804 -> TLV9302; Digikey LT1804CS8#PBF-ND -> 296-53513-1-ND; MPN (none) -> TLV9302IDR; Manufacturer (none) -> Texas Instruments

Commit message: Running DRC on PCB
Parts:
- J3, J4: value Conn_01x02_Socket -> 0022272021
Changed lines of the file:
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@@
 			)
 		)
-		(property "Value" "Conn_01x02_Socket"
+		(property "Value" "0022272021"
 			(at 38.1 35.5599 0)
 			(effects
@@
 			)
 		)
-		(property "Value" "Conn_01x02_Socket"
+		(property "Value" "0022272021"
 			(at 269.24 134.6199 0)
 			(effects

Commit message: Adding gerbers and bom for gate driver
Other:
- company: (none) -> openEPR
- title: (none) -> Drain Driver
Changed lines of the file:
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@@
 	(paper "A4")
 	(title_block
-		(date "2025-07-05")
-		(rev "1.1")
+		(title "Drain Driver")
+		(date "2025-07-11")
+		(rev "3.0")
+		(company "openEPR")
 	)
 	(rectangle

Commit message: Adding notes to schematic
Parts:
- added C25, C28, C29, C30: 100nF, Capacitor_SMD:C_0805_2012Metric, symbol Device:C_Small
- added C26, C27: 10uF, Capacitor_SMD:C_0805_2012Metric, symbol Device:C_Small
Connections:
- net GND: now also C25.1, C26.2, C27.2, C28.1, C29.1, C30.1
- net VCC: now also C25.2, C26.1, C27.1, C28.2, C29.2, C30.2
Other:
- moved on the sheet: C11, C12, C14, C9, J3
