File: Hardware/X-Band Amplifier QPA1022/X-Band Amplifier QPA1022.kicad_pcb (KiCad board)
At the start: 4 copper layers, 25.4 x 25.4 mm, 15 parts, among them J1 901-10513-3, J2 901-10513-3, U1 QPA1022

Commit message: Updating 4W amplifier, creating gerbers
Routing:
- net GND: vias 179 -> 223
Other:
- board text added: "0.2104mm Thick FR4 Dr = 4.4 JLC04161H-7628 W = 0.4mm S = 0.4mm Z0 = 50 ohm"
- board text added: "4W AMP"
- board text added: "QPA1022"
