File: Hardware/AFC/input_stage.kicad_sch (KiCad schematic)
At the start: 61 parts, among them J2 Conn_Coaxial, J3 Conn_Coaxial, J8 Conn_Coaxial, U1 AD633JRZ, U13 AD8676xR, U2 AD633JRZ, U4 AD8676xR, U6 LM358, U8 LM358

Commit message: Minor Changes
Other:
- note added: "Consider NE5532 low noise op amp as a replacement."
Changed lines of the file:
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@@
 	(text "Cross Term AFC\n(IQ Mixer)"
 		(exclude_from_sim no)
-		(at 26.67 54.356 0)
+		(at 31.242 53.848 0)
 		(effects
 			(font
@@
 	(text "or Conventional Dispersion (Q^{2} only)"
 		(exclude_from_sim no)
-		(at 26.67 58.928 0)
+		(at 33.274 62.738 0)
 		(effects
 			(font
+				(size 1.27 1.27)
+			)
+		)
+	)
+	(text "Consider NE5532 low noise op amp as a replacement."
+		(exclude_from_sim no)
+		(at 168.656 20.066 0)
+		(effects
+			(font
