File: Hardware/S-Band LGR Void/S-Band LGR Void.kicad_pcb (KiCad board)
At the start: 2 copper layers, 38 x 20.1 mm, 7 parts

Commit message: Updates to LGR Void
Parts:
- removed C1, C2: 0.2pF, Capacitor_SMD:C_0402_1005Metric
- AE1: footprint _tim-RF:LGR_5.2mm -> _tim-RF:LGR_Void_10mm
