File: Hardware/S-Band LGR Void/S-Band LGR Void.kicad_sch (KiCad schematic)
At the start: 5 parts

Commit message: Updates to LGR Void
Parts:
- AE1: footprint _tim-RF:LGR_5.2mm -> _tim-RF:LGR_Void_10mm
Changed lines of the file:
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@@
 			)
 		)
-		(property "Footprint" "_tim-RF:LGR_5.2mm"
+		(property "Footprint" "_tim-RF:LGR_Void_10mm"
 			(at 114.3 33.02 0)
 			(effects
