File: Hardware/S-Band Circulator/S-Band Circulator.kicad_pcb (KiCad board)
At the start: 4 copper layers, 38.1 x 25.4 mm, 8 parts, among them J1 SMA-J-P-H-ST-EM1, J2 SMA-J-P-H-ST-EM1, J3 SMA-J-P-H-ST-EM1, U1 0735912050

Commit message: Adding Gerbers
Changed lines of the file:
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@@
 			(outputformat 1)
 			(mirror no)
-			(drillshape 1)
+			(drillshape 0)
 			(scaleselection 1)
-			(outputdirectory "")
+			(outputdirectory "${PROJECTNAME}_${REVISION}_Gerbers")
 		)
 	)
@@
 			(font
 				(size 1 1)
-				(thickness 0.1)
+				(thickness 0.15)
 			)
 			(justify bottom)
@@
 			(keep_text_aligned yes)
 		)
-		(gr_text "1.5"
+		(gr_text "38.1"
 			(at 95.25 19.805 0)
 			(layer "Dwgs.User")
@@
 			(keep_text_aligned yes)
 		)
-		(gr_text "1.2"
+		(gr_text "30.48"
 			(at 95.25 22.98 0)
 			(layer "Dwgs.User")
