File: Hardware/S-Band Limiter/S-Band Limiter.kicad_pcb (KiCad board)
At the start: 4 copper layers, 35 x 25 mm, 11 parts, among them J1 SMA-J-P-H-ST-EM1, J2 SMA-J-P-H-ST-EM1, U1 SKY16603-632LF, U2 CLA4607-085LF

Commit message: Adding Gerbers
Parts:
- C1, C2: value 18pF -> 22pF
Changed lines of the file:
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@@
 			(outputformat 1)
 			(mirror no)
-			(drillshape 1)
+			(drillshape 0)
 			(scaleselection 1)
-			(outputdirectory "")
+			(outputdirectory "${PROJECTNAME}_${REVISION}_Gerbers")
 		)
 	)
@@
 			)
 		)
-		(property "Value" "18pF"
+		(property "Value" "22pF"
 			(at 0 1.16 0)
 			(layer "F.Fab")
@@
 			)
 		)
-		(property "Value" "18pF"
+		(property "Value" "22pF"
 			(at 0 1.16 0)
 			(layer "F.Fab")
@@
 		(tags "inductor")
 		(property "Reference" "L1"
-			(at 2.1566 0 90)
+			(at 2.1566 0 0)
 			(layer "F.SilkS")
 			(effects
@@
 			(font
 				(size 1 1)
-				(thickness 0.1)
+				(thickness 0.15)
 			)
 			(justify bottom)
@@
 			(keep_text_aligned yes)
 		)
-		(gr_text "0.7087"
+		(gr_text "18"
 			(at 116.35 40 90)
 			(layer "Dwgs.User")
@@
 			(keep_text_aligned yes)
 		)
-		(gr_text "0.9843"
+		(gr_text "25"
 			(at 118.85 40 90)
 			(layer "Dwgs.User")
@@
 			(keep_text_aligned yes)
 		)
-		(gr_text "1.378"
+		(gr_text "35"
 			(at 97.5 22.85 0)
 			(layer "Dwgs.User")
@@
 			(keep_text_aligned yes)
 		)
-		(gr_text "1.1024"
+		(gr_text "28"
 			(at 97.5 25.35 0)
 			(layer "Dwgs.User")
