File: Hardware/S-Band Limiter/S-Band Limiter.kicad_sch (KiCad schematic)
At the start: 11 parts, among them J1 SMA-J-P-H-ST-EM1, J2 SMA-J-P-H-ST-EM1, U1 SKY16603-632LF, U2 CLA4607-085LF

Commit message: Adding Gerbers
Parts:
- C1, C2: value 18pF -> 22pF
Changed lines of the file:
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@@
 			)
 		)
-		(property "Value" "18pF"
+		(property "Value" "22pF"
 			(at 104.1463 43.18 90)
 			(effects
@@
 			)
 		)
-		(property "Value" "18pF"
+		(property "Value" "22pF"
 			(at 67.3163 43.18 90)
 			(effects
