File: Hardware/Phase_shifter_150MHz/Phase_shifter_150MHz.kicad_pcb (KiCad board)
At the start: 2 copper layers, 60 x 50 mm, 22 parts, among them J1 0022272021, J2 SMA-J-P-H-ST-EM1, J3 SMA-J-P-H-ST-EM1, J4 SMA-J-P-H-ST-EM1, U1 LM358, U2 SCPHS-180+

Commit message: Adding Gerbers
Parts:
- moved J1 2.55 mm to (105.8, 66.3), turned to 90 degrees
- moved C1 0.25 mm to (92.2, 60.5)
- moved C3 0.25 mm to (67.8, 65.5)
- moved C4 0.25 mm to (67.8, 62.9)
- moved R3 0.25 mm to (67.8, 60.5)
- moved R4 0.25 mm to (92.2, 63.0)
Routing:
- net +12V: track 19.0 -> 27.4 mm
- net GND: vias 91 -> 94
Other:
- board text added: "+12V"
- board text added: "BIAS +5V MAX"
- board text added: "GND"
- board text added: "RF IN"
- board text added: "RF OUT"
